Commit message: Complete Collision and visual

File: src/mark1_description/urdf/mark1 (copy).xacro (robot description, xacro)
@@ -16,5 +16,5 @@
       />
     </inertial>
-    <collision name='collision'>
+    <collision name='chassis_collision'>
       <origin xyz="299 195.4 211.8" rpy=" 0 0 0"/>
       <geometry>
@@ -30,6 +30,8 @@
   </link>
 <!-- Patas del rover, rocker es la larga, boogie la unida de dos ruedas /-->
+  <!-- Rocker de ambas patas, es decir las de atras /-->
   <link name="right_leg_rocker">
-    <visual name="r_up_part">
+    <!-- visual /-->
+    <visual name="r_up_part_visual">
       <geometry>
         <box size="219.5 25.4 25.4"/>
@@ -37,5 +39,5 @@
       <origin rpy="0 0 0" xyz="308.59 82.7 211.79"/>
     </visual>
-    <visual name="r_down_part">
+    <visual name="r_down_part_visual">
       <geometry>
         <box size="225 25.4 25.4"/>
@@ -43,5 +45,5 @@
       <origin rpy="0 -0.78 0" xyz="119.54 82.7 82.5"/>
     </visual>
-    <visual name="r_front_part">
+    <visual name="r_front_part_visual">
       <geometry>
         <box size="56 25.4 25.4"/>
@@ -49,7 +51,27 @@
       <origin rpy="0 0.78 0" xyz="437.89 82.7 179.3"/>
     </visual>
+    <!-- collision /-->
+    <collision name="r_up_part_collision">
+      <geometry>
+        <box size="219.5 25.4 25.4"/>
+      </geometry>
+      <origin rpy="0 0 0" xyz="308.59 82.7 211.79"/>
+    </collision>
+    <collision name="r_down_part_collision">
+      <geometry>
+        <box size="225 25.4 25.4"/>
+      </geometry>
+      <origin rpy="0 -0.78 0" xyz="119.54 82.7 82.5"/>
+    </collision>
+    <collision name="r_front_part_collision">
+      <geometry>
+        <box size="56 25.4 25.4"/>
+      </geometry>
+      <origin rpy="0 0.78 0" xyz="437.89 82.7 179.3"/>
+    </collision>
   </link>
   <link name="left_leg_rocker">
-    <visual name="l_up_part">
+    <!-- visual /-->
+    <visual name="l_up_part_visual">
       <geometry>
         <box size="219.5 25.4 25.4"/>
@@ -57,44 +79,203 @@
       <origin rpy="0 0 0" xyz="308.59 348.1 211.79"/>
     </visual>
-    <visual name="l_down_part">
-      <geometry>
-        <box size="219.5 25.4 25.4"/>
-      </geometry>
-      <origin rpy="0 -0.78 0" xyz="308.59 348.1 211.79"/>
-    </visual>
-    <visual name="l_front_part">
-      <geometry>
-        <box size="219.5 25.4 25.4"/>
-      </geometry>
-      <origin rpy="0 -0.78 0" xyz="308.59 348.1 211.79"/>
-    </visual>
-  </link>
+    <visual name="l_down_part_visual">
+      <geometry>
+        <box size="219.5 25.4 25.4"/>
+      </geometry>
+      <origin rpy="0 -0.78 0" xyz="308.59 348.1 211.79"/>
+    </visual>
+    <visual name="l_front_part_visual">
+      <geometry>
+        <box size="219.5 25.4 25.4"/>
+      </geometry>
+      <origin rpy="0 -0.78 0" xyz="308.59 348.1 211.79"/>
+    </visual>
+    <!-- collision	 /-->
+    <collision name="l_up_part_collision">
+      <geometry>
+        <box size="219.5 25.4 25.4"/>
+      </geometry>
+      <origin rpy="0 0 0" xyz="308.59 348.1 211.79"/>
+    </collision>
+    <collision name="l_down_part_collision">
+      <geometry>
+        <box size="219.5 25.4 25.4"/>
+      </geometry>
+      <origin rpy="0 -0.78 0" xyz="308.59 348.1 211.79"/>
+    </collision>
+    <collision name="l_front_part_collision">
+      <geometry>
+        <box size="219.5 25.4 25.4"/>
+      </geometry>
+      <origin rpy="0 -0.78 0" xyz="308.59 348.1 211.79"/>
+    </collision>
+  </link>
+  <!-- Boogie de ambas patas, es decir las de atras /-->
   <link name="right_leg_boogie">
-    <visual name="r_up_part_rocker">
-      <geometry>
-        <box size="219.5 25.4 25.4"/>
-      </geometry>
-      <origin rpy="0 0 0" xyz="308.59 82.7 211.79"/>
-    </visual>
-    <visual name="r_down_part">
-      <geometry>
-        <box size="219.5 25.4 25.4"/>
-      </geometry>
-      <origin rpy="0 -0.78 0" xyz="308.59 82.7 211.79"/>
-    </visual>
-  </link>
-  <link name="left_leg_rocker">
-    <visual name="l_up_part">
-      <geometry>
-        <box size="219.5 25.4 25.4"/>
-      </geometry>
-      <origin rpy="0 0 0" xyz="308.59 348.1 211.79"/>
-    </visual>
-    <visual name="l_down_part">
-      <geometry>
-        <box size="219.5 25.4 25.4"/>
-      </geometry>
-      <origin rpy="0 -0.78 0" xyz="308.59 348.1 211.79"/>
-    </visual>
+    <!-- visual /-->
+    <visual name="r_base_visual">
+      <geometry>
+        <box size="40.0 25.4 25.4"/>
+      </geometry>
+      <origin rpy="0 0 0" xyz="438.0 82.7 172.2"/>
+    </visual>
+    <visual name="r_front_visual">
+      <geometry>
+        <box size="25.4 119.5 25.4"/>
+      </geometry>
+      <origin rpy="0 0 0" xyz="470.7 82.7 99.75"/>
+    </visual>
+    <visual name="r_back_visual">
+      <geometry>
+        <box size="25.4 119.5 25.4"/>
+      </geometry>
+      <origin rpy="0 0 0" xyz="405.3 82.7 99.75"/>
+    </visual>
+    <!-- collision /-->
+    <collision name="r_base_collision">
+      <geometry>
+        <box size="40.0 25.4 25.4"/>
+      </geometry>
+      <origin rpy="0 0 0" xyz="438.0 82.7 172.2"/>
+    </collision>
+    <collision name="r_front_collision">
+      <geometry>
+        <box size="25.4 119.5 25.4"/>
+      </geometry>
+      <origin rpy="0 0 0" xyz="470.7 82.7 99.75"/>
+    </collision>
+    <collision name="r_back_collision">
+      <geometry>
+        <box size="25.4 119.5 25.4"/>
+      </geometry>
+      <origin rpy="0 0 0" xyz="405.3 82.7 99.75"/>
+    </collision>
+  </link>
+  <link name="left_leg_boogie">
+    <!-- visual /-->
+    <visual name="l_base_visual">
+      <geometry>
+        <box size="40.0 25.4 25.4"/>
+      </geometry>
+      <origin rpy="0 0 0" xyz="438.0 348.1 172.2"/>
+    </visual>
+    <visual name="l_front_visual">
+      <geometry>
+        <box size="25.4 119.5 25.4"/>
+      </geometry>
+      <origin rpy="0 0 0" xyz="470.7 348.1 99.75"/>
+    </visual>
+    <visual name="l_back_visual">
+      <geometry>
+        <box size="25.4 119.5 25.4"/>
+      </geometry>
+      <origin rpy="0 0 0" xyz="405.3 348.1 99.75"/>
+    </visual>
+    <!-- collision	 /-->
+    <collision name="l_base_collision">
+      <geometry>
+        <box size="40.0 25.4 25.4"/>
+      </geometry>
+      <origin rpy="0 0 0" xyz="438.0 348.1 172.2"/>
+    </collision>
+    <collision name="l_front_collision">
+      <geometry>
+        <box size="25.4 119.5 25.4"/>
+      </geometry>
+      <origin rpy="0 0 0" xyz="470.7 348.1 99.75"/>
+    </collision>
+    <collision name="l_back_collision">
+      <geometry>
+        <box size="25.4 119.5 25.4"/>
+      </geometry>
+      <origin rpy="0 0 0" xyz="405.3 348.1 99.75"/>
+    </collision>
+  </link>
+  <!--Llantas, son 6 en total 3 a cada lado  ..................... /-->
+  <!--Llantas derechas/-->
+  <link name="right_wheel_front">
+    <visual name="right_wheel_front_visual">
+      <origin rpy="0 1.5707 1.5707" xyz="40.0 25.0 40.0"/>
+      <geometry>
+        <cylinder length="50.0" radius="40.0"/>
+      </geometry>
+    </visual>
+    <collision name="right_wheel_front_collision">
+      <origin rpy="0 1.5707 1.5707" xyz="40.0 25.0 40.0"/>
+      <geometry>
+        <cylinder length="50.0" radius="40.0"/>
+      </geometry>
+    </collision>
+  </link>
+  <link name="right_wheel_medium">
+    <visual name="right_wheel_medium_visual">
+      <origin rpy="0 1.5707 1.5707" xyz="418.0 25.0 40.0"/>
+      <geometry>
+        <cylinder length="50.0" radius="40.0"/>
+      </geometry>
+    </visual>
+    <collision name="right_wheel_medium_collision">
+      <origin rpy="0 1.5707 1.5707" xyz="418.0 25.0 40.0"/>
+      <geometry>
+        <cylinder length="50.0" radius="40.0"/>
+      </geometry>
+    </collision>
+  </link>
+  <link name="right_wheel_back">
+    <visual name="right_wheel_back_visual">
+      <origin rpy="0 1.5707 1.5707" xyz="458.0 25.0 40.0"/>
+      <geometry>
+        <cylinder length="50.0" radius="40.0"/>
+      </geometry>
+    </visual>
+    <collision name="right_wheel_back_collision">
+      <origin rpy="0 1.5707 1.5707" xyz="458.0 25.0 40.0"/>
+      <geometry>
+        <cylinder length="50.0" radius="40.0"/>
+      </geometry>
+    </collision>
+  </link>
+  <!--Llantas izquierdas/-->
+  <link name="left_wheel_front">
+    <visual name="left_wheel_front_visual">
+      <origin rpy="0 1.5707 1.5707" xyz="40.0 405.8 40.0"/>
+      <geometry>
+        <cylinder length="50.0" radius="40.0"/>
+      </geometry>
+    </visual>
+    <collision name="left_wheel_front_collision">
+      <origin rpy="0 1.5707 1.5707" xyz="40.0 405.8 40.0"/>
+      <geometry>
+        <cylinder length="50.0" radius="40.0"/>
+      </geometry>
+    </collision>
+  </link>
+  <link name="left_wheel_medium">
+    <visual name="left_wheel_medium_visual">
+      <origin rpy="0 1.5707 1.5707" xyz="418.0 405.8 40.0"/>
+      <geometry>
+        <cylinder length="50.0" radius="40.0"/>
+      </geometry>
+    </visual>
+    <collision name="left_wheel_medium_collision">
+      <origin rpy="0 1.5707 1.5707" xyz="418.0 405.8 40.0"/>
+      <geometry>
+        <cylinder length="50.0" radius="40.0"/>
+      </geometry>
+    </collision>
+  </link>
+  <link name="left_wheel_back">
+    <visual name="left_wheel_back_visual">
+      <origin rpy="0 1.5707 1.5707" xyz="458.0 405.8 40.0"/>
+      <geometry>
+        <cylinder length="50.0" radius="40.0"/>
+      </geometry>
+    </visual>
+    <collision name="left_wheel_back_collision">
+      <origin rpy="0 1.5707 1.5707" xyz="458.0 405.8 40.0"/>
+      <geometry>
+        <cylinder length="50.0" radius="40.0"/>
+      </geometry>
+    </collision>
   </link>
 <!-- estos valores no se si sirve/-->

Commit message: Fixed complete scale

File: src/mark1_description/urdf/mark1 (copy).xacro (robot description, xacro)
@@ -5,9 +5,9 @@
 <!-- Chassis, caja de control /-->
 <link name='chassis'>
-    <pose>299 195.4 211.8 0 0 0</pose >
+    <pose>0.299 0.1954 0.2118 0 0 0</pose >
 <!-- estos valores no se si sirve/-->
     <inertial>
       <mass value="4"/>
-      <origin xyz="299.0 195.4 211.8" rpy=" 0 0 0"/>
+      <origin xyz="0.2990 0.1954 0.2118" rpy=" 0 0 0"/>
       <inertia
           ixx="0.0001" ixy="0" ixz="0"
@@ -17,13 +17,13 @@
     </inertial>
     <collision name='chassis_collision'>
-      <origin xyz="299 195.4 211.8" rpy=" 0 0 0"/>
-      <geometry>
-        <box size="200.0 200.0 100.0"/>
+      <origin xyz="0.299 0.1954 0.2118" rpy=" 0 0 0"/>
+      <geometry>
+        <box size="0.2000 0.2000 0.1000"/>
       </geometry>
     </collision>
     <visual name='chassis_visual'>
-      <origin xyz="299 195.4 211.8" rpy=" 0 0 0"/>
-      <geometry>
-        <box size="200.0 200.0 100.0"/>
+      <origin xyz="0.299 0.1954 0.2118" rpy=" 0 0 0"/>
+      <geometry>
+        <box size="0.02000 0.0200 0.01000"/>
       </geometry>
     </visual>
@@ -35,32 +35,32 @@
     <visual name="r_up_part_visual">
       <geometry>
-        <box size="219.5 25.4 25.4"/>
-      </geometry>
-      <origin rpy="0 0 0" xyz="308.59 82.7 211.79"/>
+        <box size="0.2195 0.00254 0.00254"/>
+      </geometry>
+      <origin rpy="0 0 0" xyz="0.30859 0.0827 0.021179"/>
     </visual>
     <visual name="r_down_part_visual">
       <geometry>
-        <box size="225 25.4 25.4"/>
-      </geometry>
-      <origin rpy="0 -0.78 0" xyz="119.54 82.7 82.5"/>
+        <box size="0.225 0.00254 0.00254"/>
+      </geometry>
+      <origin rpy="0 -0.78 0" xyz="0.11954 0.0827 0.0825"/>
     </visual>
     <visual name="r_front_part_visual">
       <geometry>
-        <box size="56 25.4 25.4"/>
-      </geometry>
-      <origin rpy="0 0.78 0" xyz="437.89 82.7 179.3"/>
+        <box size="0.056 0.00254 0.00254"/>
+      </geometry>
+      <origin rpy="0 0.78 0" xyz="0.43789 0.0827 0.1793"/>
     </visual>
     <!-- collision /-->
     <collision name="r_up_part_collision">
       <geometry>
-        <box size="219.5 25.4 25.4"/>
-      </geometry>
-      <origin rpy="0 0 0" xyz="308.59 82.7 211.79"/>
+        <box size="0.2195 0.00254 0.00254"/>
+      </geometry>
+      <origin rpy="0 0 0" xyz="0.30859 0.0827 0.21179"/>
     </collision>
     <collision name="r_down_part_collision">
       <geometry>
-        <box size="225 25.4 25.4"/>
-      </geometry>
-      <origin rpy="0 -0.78 0" xyz="119.54 82.7 82.5"/>
+        <box size="0.225 0.00254 0.00254"/>
+      </geometry>
+      <origin rpy="0 -0.78 0" xyz="0.11954 0.0827 0.0825"/>
     </collision>
     <collision name="r_front_part_collision">
@@ -75,40 +75,41 @@
     <visual name="l_up_part_visual">
       <geometry>
-        <box size="219.5 25.4 25.4"/>
-      </geometry>
-      <origin rpy="0 0 0" xyz="308.59 348.1 211.79"/>
+        <box size="0.2195 0.00254 0.00254"/>
+      </geometry>
+      <origin rpy="0 0 0" xyz="0.30859 0.3481 0.21179"/>
     </visual>
     <visual name="l_down_part_visual">
       <geometry>
-        <box size="219.5 25.4 25.4"/>
-      </geometry>
-      <origin rpy="0 -0.78 0" xyz="308.59 348.1 211.79"/>
+        <box size="0.2195 0.00254 0.00254"/>
+      </geometry>
+      <origin rpy="0 -0.78 0" xyz="0.30859 0.3481 0.21179"/>
     </visual>
     <visual name="l_front_part_visual">
       <geometry>
-        <box size="219.5 25.4 25.4"/>
-      </geometry>
-      <origin rpy="0 -0.78 0" xyz="308.59 348.1 211.79"/>
+        <box size="0.2195 0.00254 0.00254"/>
+      </geometry>
+      <origin rpy="0 -0.78 0" xyz="0.30859 0.3481 0.21179"/>
     </visual>
     <!-- collision	 /-->
     <collision name="l_up_part_collision">
       <geometry>
-        <box size="219.5 25.4 25.4"/>
-      </geometry>
-      <origin rpy="0 0 0" xyz="308.59 348.1 211.79"/>
+        <box size="0.2195 0.00254 0.00254"/>
+      </geometry>
+      <origin rpy="0 0 0" xyz="0.30859 0.3481 0.21179"/>
     </collision>
     <collision name="l_down_part_collision">
       <geometry>
-        <box size="219.5 25.4 25.4"/>
-      </geometry>
-      <origin rpy="0 -0.78 0" xyz="308.59 348.1 211.79"/>
+        <box size="0.2195 0.00254 0.00254"/>
+      </geometry>
+      <origin rpy="0 -0.78 0" xyz="0.30859 0.3481 0.21179"/>
     </collision>
     <collision name="l_front_part_collision">
       <geometry>
-        <box size="219.5 25.4 25.4"/>
-      </geometry>
-      <origin rpy="0 -0.78 0" xyz="308.59 348.1 211.79"/>
-    </collision>
-  </link>
+        <box size="0.2195 0.254 0.254"/>
+      </geometry>
+      <origin rpy="0 -0.78 0" xyz="0.30859 0.3481 0.21179"/>
+    </collision>
+  </link>
+-
   <!-- Boogie de ambas patas, es decir las de atras /-->
   <link name="right_leg_boogie">
@@ -116,38 +117,38 @@
     <visual name="r_base_visual">
       <geometry>
-        <box size="40.0 25.4 25.4"/>
-      </geometry>
-      <origin rpy="0 0 0" xyz="438.0 82.7 172.2"/>
+        <box size="0.0400 0.00254 0.00254"/>
+      </geometry>
+      <origin rpy="0 0 0" xyz="0.4380 0.0827 0.1722"/>
     </visual>
     <visual name="r_front_visual">
       <geometry>
-        <box size="25.4 119.5 25.4"/>
-      </geometry>
-      <origin rpy="0 0 0" xyz="470.7 82.7 99.75"/>
+        <box size="0.00254 0.1195 0.00254"/>
+      </geometry>
+      <origin rpy="0 0 0" xyz="0.4707 0.0827 0.09975"/>
     </visual>
     <visual name="r_back_visual">
       <geometry>
-        <box size="25.4 119.5 25.4"/>
-      </geometry>
-      <origin rpy="0 0 0" xyz="405.3 82.7 99.75"/>
+        <box size="0.00254 0.1195 0.00254"/>
+      </geometry>
+      <origin rpy="0 0 0" xyz="0.4053 0.0827 0.09975"/>
     </visual>
     <!-- collision /-->
-    <collision name="r_base_collision">
-      <geometry>
-        <box size="40.0 25.4 25.4"/>
-      </geometry>
-      <origin rpy="0 0 0" xyz="438.0 82.7 172.2"/>
+<collision name="r_base_collision">
+      <geometry>
+        <box size="0.400 0.00254 0.00254"/>
+      </geometry>
+      <origin rpy="0 0 0" xyz="0.4380 0.0827 0.1722"/>
     </collision>
     <collision name="r_front_collision">
       <geometry>
-        <box size="25.4 119.5 25.4"/>
-      </geometry>
-      <origin rpy="0 0 0" xyz="470.7 82.7 99.75"/>
+        <box size="0.00254 0.01195 0.00254"/>
+      </geometry>
+      <origin rpy="0 0 0" xyz="0.04707 0.0827 0.09975"/>
     </collision>
     <collision name="r_back_collision">
       <geometry>
-        <box size="25.4 119.5 25.4"/>
-      </geometry>
-      <origin rpy="0 0 0" xyz="405.3 82.7 99.75"/>
+        <box size="0.00254 0.1195 0.00254"/>
+      </geometry>
+      <origin rpy="0 0 0" xyz="0.4053 0.0827 0.09975"/>
     </collision>
   </link>
@@ -156,38 +157,38 @@
     <visual name="l_base_visual">
       <geometry>
-        <box size="40.0 25.4 25.4"/>
-      </geometry>
-      <origin rpy="0 0 0" xyz="438.0 348.1 172.2"/>
+        <box size="0.0400 0.00254 0.00254"/>
+      </geometry>
+      <origin rpy="0 0 0" xyz="0.4380 0.3481 0.1722"/>
     </visual>
     <visual name="l_front_visual">
       <geometry>
-        <box size="25.4 119.5 25.4"/>
-      </geometry>
-      <origin rpy="0 0 0" xyz="470.7 348.1 99.75"/>
+        <box size="0.00254 0.1195 0.00254"/>
+      </geometry>
+      <origin rpy="0 0 0" xyz="0.4707 0.3481 0.09975"/>
     </visual>
     <visual name="l_back_visual">
       <geometry>
-        <box size="25.4 119.5 25.4"/>
-      </geometry>
-      <origin rpy="0 0 0" xyz="405.3 348.1 99.75"/>
+        <box size="0.00254 0.1195 0.00254"/>
+      </geometry>
+      <origin rpy="0 0 0" xyz="0.4053 0.3481 0.09975"/>
     </visual>
     <!-- collision	 /-->
     <collision name="l_base_collision">
       <geometry>
-        <box size="40.0 25.4 25.4"/>
-      </geometry>
-      <origin rpy="0 0 0" xyz="438.0 348.1 172.2"/>
+        <box size="0.400 0.00254 0.00254"/>
+      </geometry>
+      <origin rpy="0 0 0" xyz="0.4380 0.3481 0.1722"/>
     </collision>
     <collision name="l_front_collision">
       <geometry>
-        <box size="25.4 119.5 25.4"/>
-      </geometry>
-      <origin rpy="0 0 0" xyz="470.7 348.1 99.75"/>
+        <box size="0.00254 0.1195 0.00254"/>
+      </geometry>
+      <origin rpy="0 0 0" xyz="0.4707 0.3481 0.09975"/>
     </collision>
     <collision name="l_back_collision">
       <geometry>
-        <box size="25.4 119.5 25.4"/>
-      </geometry>
-      <origin rpy="0 0 0" xyz="405.3 348.1 99.75"/>
+        <box size="0.00254 0.1195 0.00254"/>
+      </geometry>
+      <origin rpy="0 0 0" xyz="0.4053 0.3481 0.09975"/>
     </collision>
   </link>
@@ -196,13 +197,13 @@
   <link name="right_wheel_front">
     <visual name="right_wheel_front_visual">
-      <origin rpy="0 1.5707 1.5707" xyz="40.0 25.0 40.0"/>
-      <geometry>
-        <cylinder length="50.0" radius="40.0"/>
+      <origin rpy="0 1.5707 1.5707" xyz="0.00400 0.00250 0.00400"/>
+      <geometry>
+        <cylinder length="0.00500" radius="0.00400"/>
       </geometry>
     </visual>
     <collision name="right_wheel_front_collision">
-      <origin rpy="0 1.5707 1.5707" xyz="40.0 25.0 40.0"/>
-      <geometry>
-        <cylinder length="50.0" radius="40.0"/>
+      <origin rpy="0 1.5707 1.5707" xyz="0.00400 0.00250 0.00400"/>
+      <geometry>
+        <cylinder length="0.00500" radius="0.00400"/>
       </geometry>
     </collision>
@@ -210,13 +211,13 @@
   <link name="right_wheel_medium">
     <visual name="right_wheel_medium_visual">
-      <origin rpy="0 1.5707 1.5707" xyz="418.0 25.0 40.0"/>
-      <geometry>
-        <cylinder length="50.0" radius="40.0"/>
+      <origin rpy="0 1.5707 1.5707" xyz="0.4180 0.00250 0.00400"/>
+      <geometry>
+        <cylinder length="0.00500" radius="0.00400"/>
       </geometry>
     </visual>
     <collision name="right_wheel_medium_collision">
-      <origin rpy="0 1.5707 1.5707" xyz="418.0 25.0 40.0"/>
-      <geometry>
-        <cylinder length="50.0" radius="40.0"/>
+      <origin rpy="0 1.5707 1.5707" xyz="0.4180 0.00250 0.00400"/>
+      <geometry>
+        <cylinder length="0.00500" radius="0.00400"/>
       </geometry>
     </collision>
@@ -224,13 +225,13 @@
   <link name="right_wheel_back">
     <visual name="right_wheel_back_visual">
-      <origin rpy="0 1.5707 1.5707" xyz="458.0 25.0 40.0"/>
-      <geometry>
-        <cylinder length="50.0" radius="40.0"/>
+      <origin rpy="0 1.5707 1.5707" xyz="0.4580 0.00250 0.00400"/>
+      <geometry>
+        <cylinder length="0.00500" radius="0.00400"/>
       </geometry>
     </visual>
     <collision name="right_wheel_back_collision">
-      <origin rpy="0 1.5707 1.5707" xyz="458.0 25.0 40.0"/>
-      <geometry>
-        <cylinder length="50.0" radius="40.0"/>
+      <origin rpy="0 1.5707 1.5707" xyz="0.4580 0.00250 0.00400"/>
+      <geometry>
+        <cylinder length="0.00500" radius="0.00400"/>
       </geometry>
     </collision>
@@ -239,13 +240,13 @@
   <link name="left_wheel_front">
     <visual name="left_wheel_front_visual">
-      <origin rpy="0 1.5707 1.5707" xyz="40.0 405.8 40.0"/>
-      <geometry>
-        <cylinder length="50.0" radius="40.0"/>
+      <origin rpy="0 1.5707 1.5707" xyz="0.0040.0 0.4058 0.00400"/>
+      <geometry>
+        <cylinder length="0.00500" radius="0.00400"/>
       </geometry>
     </visual>
     <collision name="left_wheel_front_collision">
-      <origin rpy="0 1.5707 1.5707" xyz="40.0 405.8 40.0"/>
-      <geometry>
-        <cylinder length="50.0" radius="40.0"/>
+      <origin rpy="0 1.5707 1.5707" xyz="0.00400 0.4058 0.00400"/>
+      <geometry>
+        <cylinder length="0.00500" radius="0.00400"/>
       </geometry>
     </collision>
@@ -253,13 +254,13 @@
   <link name="left_wheel_medium">
     <visual name="left_wheel_medium_visual">
-      <origin rpy="0 1.5707 1.5707" xyz="418.0 405.8 40.0"/>
-      <geometry>
-        <cylinder length="50.0" radius="40.0"/>
+      <origin rpy="0 1.5707 1.5707" xyz="0.4180 0.4058 0.00400"/>
+      <geometry>
+        <cylinder length="0.00500" radius="0.00400"/>
       </geometry>
     </visual>
     <collision name="left_wheel_medium_collision">
-      <origin rpy="0 1.5707 1.5707" xyz="418.0 405.8 40.0"/>
-      <geometry>
-        <cylinder length="50.0" radius="40.0"/>
+      <origin rpy="0 1.5707 1.5707" xyz="0.4180 0.4058 0.00400"/>
+      <geometry>
+        <cylinder length="0.00500" radius="0.00400"/>
       </geometry>
     </collision>
@@ -267,13 +268,13 @@
   <link name="left_wheel_back">
     <visual name="left_wheel_back_visual">
-      <origin rpy="0 1.5707 1.5707" xyz="458.0 405.8 40.0"/>
-      <geometry>
-        <cylinder length="50.0" radius="40.0"/>
+      <origin rpy="0 1.5707 1.5707" xyz="0.4580 0.4058 0.00400"/>
+      <geometry>
+        <cylinder length="0.00500" radius="0.00400"/>
       </geometry>
     </visual>
     <collision name="left_wheel_back_collision">
-      <origin rpy="0 1.5707 1.5707" xyz="458.0 405.8 40.0"/>
-      <geometry>
-        <cylinder length="50.0" radius="40.0"/>
+      <origin rpy="0 1.5707 1.5707" xyz="0.4580 0.4058 0.00400"/>
+      <geometry>
+        <cylinder length="0.00500" radius="0.00400"/>
       </geometry>
     </collision>
