Commit message: Test 1_2

File: src/mark1_description/urdf/mark1_1.xacro (robot description, xacro)
@@ -10,25 +10,25 @@
 </joint>
 <link name='chassis'>
-    <pose>299 195.4 211.8 0 0 0</pose >
+    <pose>0.299 0.1954 0.2118 0 0 0</pose >
 <!-- estos valores no se si sirve/-->
     <inertial>
       <mass value="4"/>
-      <origin xyz="299.0 195.4 211.8" rpy=" 0 0 0"/>
+      <origin xyz="0.299 0.1954 0.2118" rpy=" 0 0 0"/>
       <inertia
-          ixx="0.0001" ixy="0" ixz="0"
-          iyy="0.0001" iyz="0"
-          izz="0.0001"
+          ixx="0.01" ixy="0" ixz="0"
+          iyy="0.01" iyz="0"
+          izz="0.01"
       />
     </inertial>
     <collision name='collision'>
-      <origin xyz="299 195.4 211.8" rpy=" 0 0 0"/>
+      <origin xyz="0.299 0.1954 0.2118" rpy=" 0 0 0"/>
       <geometry>
-        <box size="200.0 200.0 100.0"/>
+        <box size="0.2000 0.2000 0.100"/>
       </geometry>
     </collision>
     <visual name='chassis_visual'>
-      <origin xyz="299 195.4 211.8" rpy=" 0 0 0"/>
+      <origin xyz="0.299 0.1954 0.2118" rpy=" 0 0 0"/>
       <geometry>
-        <box size="200.0 200.0 100.0"/>
+        <box size="0.2000 0.2000 0.100"/>
       </geometry>
       <material name="orange">
@@ -47,27 +47,27 @@
     <visual name="r_up_part">
       <geometry>
-        <box size="219.5 25.4 25.4"/>
+        <box size="0.2195 0.0254 0.0254"/>
       </geometry>
-      <origin rpy="0 0 0" xyz="308.59 82.7 211.79"/>
+      <origin rpy="0 0 0" xyz="0.30859 0.0827 0.21179"/>
     </visual>
     <visual name="r_down_part">
       <geometry>
-        <box size="225 25.4 25.4"/>
+        <box size="0.225 0.0254 0.0254"/>
       </geometry>
-      <origin rpy="0 -0.78 0" xyz="119.54 82.7 82.5"/>
+      <origin rpy="0 -0.78 0" xyz="0.11954 0.0827 0.0825"/>
     </visual>
     <visual name="r_front_part">
       <geometry>
-        <box size="56 25.4 25.4"/>
+        <box size="0.056 0.0254 0.0254"/>
       </geometry>
-      <origin rpy="0 0.78 0" xyz="437.89 82.7 179.3"/>
+      <origin rpy="0 0.78 0" xyz="0.43789 0.0827 0.1793"/>
     </visual>
     <inertial>
-      <mass value="1"/>
-      <origin rpy="0 -0.78 0" xyz="308.59 82.7 211.79"/>
+      <mass value="2"/>
+      <origin rpy="0 -0.78 0" xyz="0.30859 0.0827 0.21179"/>
       <inertia
-          ixx="0.0001" ixy="0" ixz="0"
-          iyy="0.0001" iyz="0"
-          izz="0.0001"
+          ixx="0.01" ixy="0" ixz="0"
+          iyy="0.1" iyz="0"
+          izz="0.01"
       />
     </inertial>
@@ -83,21 +83,21 @@
     <visual name="l_up_part">
       <geometry>
-        <box size="219.5 25.4 25.4"/>
+        <box size="0.219 0.0254 0.0254"/>
       </geometry>
-      <origin rpy="0 0 0" xyz="308.59 348.1 211.79"/>
+      <origin rpy="0 0 0" xyz="0.30859 0.3481 0.21179"/>
     </visual>
     <visual name="l_down_part">
       <geometry>
-        <box size="219.5 25.4 25.4"/>
+        <box size="0.2195 0.0254 0.0254"/>
       </geometry>
-      <origin rpy="0 -0.78 0" xyz="308.59 348.1 211.79"/>
+      <origin rpy="0 -0.78 0" xyz="0.30859 0.3481 0.21179"/>
     </visual>
     <inertial>
-      <mass value="1"/>
-      <origin rpy="0 -0.78 0" xyz="308.59 348.1 211.79"/>
+      <mass value="2"/>
+      <origin rpy="0 -0.78 0" xyz="0.30859 0.3481 0.21179"/>
       <inertia
-          ixx="0.0001" ixy="0" ixz="0"
-          iyy="0.0001" iyz="0"
-          izz="0.0001"
+          ixx="0.01" ixy="0" ixz="0"
+          iyy="0.01" iyz="0"
+          izz="0.01"
       />
     </inertial>
