Commit message: joint

File: src/mark1_description/urdf/mark1(copy).xacro (robot description, xacro)
@@ -3,31 +3,44 @@
   <!--xacro:include filename="$(find astromech_description)/urdf/materials.xacro" /-->
   <!--xacro:include filename="$(find astromech_description)/urdf/macros.xacro"/-->
-<!-- Chassis, caja de control /-->
-<link name='chassis'>
-    <pose>0.299 0.1954 0.2118 0 0 0</pose >
-<!-- estos valores no se si sirve/-->
-    <inertial>
-      <mass value="4"/>
-      <origin xyz="0.2990 0.1954 0.2118" rpy=" 0 0 0"/>
-      <inertia
-          ixx="0.0001" ixy="0" ixz="0"
-          iyy="0.0001" iyz="0"
-          izz="0.0001"
-      />
-    </inertial>
-    <collision name='chassis_collision'>
-      <origin xyz="0.299 0.1954 0.2118" rpy=" 0 0 0"/>
-      <geometry>
-        <box size="0.2000 0.2000 0.1000"/>
-      </geometry>
-    </collision>
-    <visual name='chassis_visual'>
-      <origin xyz="0.299 0.1954 0.2118" rpy=" 0 0 0"/>
-      <geometry>
-        <box size="0.02000 0.0200 0.01000"/>
-      </geometry>
-    </visual>
-  </link>
-<!-- Patas del rover, rocker es la larga, boogie la unida de dos ruedas /-->
+  <link name="world"></link>
+  <joint name="joint_n" type="fixed">
+    <origin xyz="0.0 0.0 0.0" rpy="0.0 0.0 0.0"/>
+    <parent link="world"/>
+    <child link="chassis"/>
+  </joint>
+  <!-- Chassis, caja de control /-->
+  <link name="chassis">
+      <pose>0.299 0.1954 0.2118 0 0 0</pose >
+    <!-- estos valores no se si sirve/-->
+      <inertial>
+        <mass value="4"/>
+        <origin xyz="0.2990 0.1954 0.2118" rpy=" 0 0 0"/>
+        <inertia
+            ixx="0.0001" ixy="0" ixz="0"
+            iyy="0.0001" iyz="0"
+            izz="0.0001"
+        />
+      </inertial>
+      <collision name='chassis_collision'>
+        <origin xyz="0.299 0.1954 0.2118" rpy=" 0 0 0"/>
+        <geometry>
+          <box size="0.2000 0.2000 0.1000"/>
+        </geometry>
+      </collision>
+      <visual name='chassis_visual'>
+        <origin xyz="0.299 0.1954 0.2118" rpy=" 0 0 0"/>
+        <geometry>
+          <box size="0.2000 0.200 0.1000"/>
+        </geometry>
+      </visual>
+  </link>
+  <joint name="joint_1" type="revolute">
+    <origin xyz="0.0 0.0 0.0" rpy="0.0 0.0 0.0"/>
+    <parent link="chassis"/>
+    <child link="right_leg_rocker"/>
+    <axis xyz="0.0 1.0 0.0"/>
+    <limit lower="0.0" upper="0.0" effort="0.0" velocity="0.0"/>
+  </joint>
+  <!-- Patas del rover, rocker es la larga, boogie la unida de dos ruedas /-->
   <!-- Rocker de ambas patas, es decir las de atras /-->
   <link name="right_leg_rocker">
@@ -71,4 +84,11 @@
     </collision>
   </link>
+  <joint name="joint_2" type="revolute">
+    <origin xyz="0.0 0.0 0.0" rpy="0.0 0.0 0.0"/>
+    <parent link="chassis"/>
+    <child link="left_leg_rocker"/>
+    <axis xyz="0.0 1.0 0.0"/>
+    <limit lower="0.0" upper="0.0" effort="0.0" velocity="0.0"/>
+  </joint>
   <link name="left_leg_rocker">
     <!-- visual /-->
@@ -111,5 +131,11 @@
     </collision>
   </link>
--
+  <joint name="joint_3" type="revolute">
+    <origin xyz="0.0 0.0 0.0" rpy="0.0 0.0 0.0"/>
+    <parent link="right_leg_rocker"/>
+    <child link="right_leg_boogie"/>
+    <axis xyz="0.0 1.0 0.0"/>
+    <limit lower="0.0" upper="0.0" effort="0.0" velocity="0.0"/>
+  </joint>
   <!-- Boogie de ambas patas, es decir las de atras /-->
   <link name="right_leg_boogie">
@@ -134,5 +160,5 @@
     </visual>
     <!-- collision /-->
-<collision name="r_base_collision">
+    <collision name="r_base_collision">
       <geometry>
         <box size="0.400 0.00254 0.00254"/>
@@ -153,4 +179,11 @@
     </collision>
   </link>
+  <joint name="joint_4" type="revolute">
+    <origin xyz="0.0 0.0 0.0" rpy="0.0 0.0 0.0"/>
+    <parent link="left_leg_rocker"/>
+    <child link="left_leg_boogie"/>
+    <axis xyz="0.0 1.0 0.0"/>
+    <limit lower="0.0" upper="0.0" effort="0.0" velocity="0.0"/>
+  </joint>
   <link name="left_leg_boogie">
     <!-- visual /-->
@@ -193,4 +226,11 @@
     </collision>
   </link>
+  <joint name="joint_5" type="revolute">
+    <origin xyz="0.0 0.0 0.0" rpy="0.0 0.0 0.0"/>
+    <parent link="right_leg_boogie"/>
+    <child link="right_wheel_front"/>
+    <axis xyz="0.0 1.0 0.0"/>
+    <limit lower="0.0" upper="0.0" effort="0.0" velocity="0.0"/>
+  </joint>
   <!--Llantas, son 6 en total 3 a cada lado  ..................... /-->
   <!--Llantas derechas/-->
@@ -209,4 +249,11 @@
     </collision>
   </link>
+  <joint name="joint_6" type="revolute">
+    <origin xyz="0.0 0.0 0.0" rpy="0.0 0.0 0.0"/>
+    <parent link="right_leg_boogie"/>
+    <child link="right_wheel_medium"/>
+    <axis xyz="0.0 1.0 0.0"/>
+    <limit lower="0.0" upper="0.0" effort="0.0" velocity="0.0"/>
+  </joint>
   <link name="right_wheel_medium">
     <visual name="right_wheel_medium_visual">
@@ -223,4 +270,11 @@
     </collision>
   </link>
+  <joint name="joint_7" type="revolute">
+    <origin xyz="0.0 0.0 0.0" rpy="0.0 0.0 0.0"/>
+    <parent link="right_leg_boogie"/>
+    <child link="right_wheel_back"/>
+    <axis xyz="0.0 1.0 0.0"/>
+    <limit lower="0.0" upper="0.0" effort="0.0" velocity="0.0"/>
+  </joint>
   <link name="right_wheel_back">
     <visual name="right_wheel_back_visual">
@@ -237,4 +291,11 @@
     </collision>
   </link>
+  <joint name="joint_8" type="revolute">
+    <origin xyz="0.0 0.0 0.0" rpy="0.0 0.0 0.0"/>
+    <parent link="left_leg_boogie"/>
+    <child link="left_wheel_front"/>
+    <axis xyz="0.0 1.0 0.0"/>
+    <limit lower="0.0" upper="0.0" effort="0.0" velocity="0.0"/>
+  </joint>
   <!--Llantas izquierdas/-->
   <link name="left_wheel_front">
@@ -252,4 +313,11 @@
     </collision>
   </link>
+  <joint name="joint_9" type="revolute">
+    <origin xyz="0.0 0.0 0.0" rpy="0.0 0.0 0.0"/>
+    <parent link="left_leg_boogie"/>
+    <child link="left_wheel_medium"/>
+    <axis xyz="0.0 1.0 0.0"/>
+    <limit lower="0.0" upper="0.0" effort="0.0" velocity="0.0"/>
+  </joint>
   <link name="left_wheel_medium">
     <visual name="left_wheel_medium_visual">
@@ -266,4 +334,11 @@
     </collision>
   </link>
+  <joint name="joint_10" type="revolute">
+    <origin xyz="0.0 0.0 0.0" rpy="0.0 0.0 0.0"/>
+    <parent link="left_leg_boogie"/>
+    <child link="left_wheel_back"/>
+    <axis xyz="0.0 1.0 0.0"/>
+    <limit lower="0.0" upper="0.0" effort="0.0" velocity="0.0"/>
+  </joint>
   <link name="left_wheel_back">
     <visual name="left_wheel_back_visual">
@@ -280,4 +355,3 @@
     </collision>
   </link>
-<!-- estos valores no se si sirve/-->
 </robot>

File: src/mark1_description/urdf/mark1_1.xacro (robot description, xacro)
@@ -5,5 +5,5 @@
 <link name='world'/>
 <joint name="joint_n" type="fixed">
-  <origin xyz="0.0 0.0 0.7" rpy="0.0 0.0 0.0"/>
+  <origin xyz="0.0 0.0 0.2" rpy="0.0 0.0 0.0"/>
   <parent link="world"/>
   <child link="chassis"/>
@@ -38,8 +38,8 @@
   </link>
   <joint name="joint_1" type="revolute">
-    <origin xyz="5 0.0 0.0" rpy="0.0 0.0 0.0"/>
+    <origin xyz="0.0 0.0 0.0" rpy="0.0 0.0 0.0"/>
     <parent link="chassis"/>
     <child link="right_leg_rocker"/>
-    <axis xyz="0.0 0.0 1.0"/>
+    <axis xyz="0.0 1.0 0.0"/>
     <limit lower="0.0" upper="0.0" effort="0.0" velocity="0.0"/>
   </joint>
@@ -47,5 +47,5 @@
     <visual name="r_up_part">
       <geometry>
-        <box size="0.2195 0.0254 0.0254"/>
+        <box size="0.2195 0.054 0.0254"/>
       </geometry>
       <origin rpy="0 0 0" xyz="0.30859 0.0827 0.21179"/>
@@ -55,5 +55,5 @@
         <box size="0.225 0.0254 0.0254"/>
       </geometry>
-      <origin rpy="0 -0.78 0" xyz="0.11954 0.0827 0.0825"/>
+      <origin rpy="0 -0.78 0" xyz="0.12954 0.0827 0.15"/>
     </visual>
     <visual name="r_front_part">
@@ -61,5 +61,5 @@
         <box size="0.056 0.0254 0.0254"/>
       </geometry>
-      <origin rpy="0 0.78 0" xyz="0.43789 0.0827 0.1793"/>
+      <origin rpy="0 0.78 0" xyz="0.42 0.0827 0.19"/>
     </visual>
     <inertial>
@@ -73,9 +73,9 @@
     </inertial>
   </link>
-  <joint name="joint_2" type="revolute">
-    <origin xyz="-5 0.0 0.0" rpy="0.0 0.0 0.0"/>
+  <joint name="joint_l" type="revolute">
+    <origin xyz="0.0 0.0 0.0" rpy="0.0 0.0 0.0"/>
     <parent link="chassis"/>
     <child link="left_leg_rocker"/>
-    <axis xyz="0.0 0.0 1.0"/>
+    <axis xyz="0.0 1.0 0.0"/>
     <limit lower="0.0" upper="0.0" effort="0.0" velocity="0.0"/>
   </joint>
@@ -83,20 +83,26 @@
     <visual name="l_up_part">
       <geometry>
-        <box size="0.219 0.0254 0.0254"/>
+        <box size="0.2195 0.054 0.0254"/>
       </geometry>
-      <origin rpy="0 0 0" xyz="0.30859 0.3481 0.21179"/>
+      <origin rpy="0 0 0" xyz="0.30859 0.2827 0.21179"/>
     </visual>
     <visual name="l_down_part">
       <geometry>
-        <box size="0.2195 0.0254 0.0254"/>
+        <box size="0.225 0.0254 0.0254"/>
       </geometry>
-      <origin rpy="0 -0.78 0" xyz="0.30859 0.3481 0.21179"/>
+      <origin rpy="0 -0.78 0" xyz="0.12954 0.2827 0.15"/>
+    </visual>
+    <visual name="l_front_part">
+      <geometry>
+        <box size="0.056 0.0254 0.0254"/>
+      </geometry>
+      <origin rpy="0 0.78 0" xyz="0.42 0.2827 0.19"/>
     </visual>
     <inertial>
       <mass value="2"/>
-      <origin rpy="0 -0.78 0" xyz="0.30859 0.3481 0.21179"/>
+      <origin rpy="0 -0.78 0" xyz="0.30859 0.2827 0.21179"/>
       <inertia
           ixx="0.01" ixy="0" ixz="0"
-          iyy="0.01" iyz="0"
+          iyy="0.1" iyz="0"
           izz="0.01"
       />

File: src/mark1_description/urdf/mark2.xacro (robot description, xacro)
@@ -1,96 +1,61 @@
 <?xml version='1.0'?>
 <robot name="mark2" xmlns:xacro="http://www.ros.org/wiki/xacro">
-    <link name='world'/>
+    <link name="world"></link>
     <joint name="joint_n" type="fixed">
-        <origin xyz="0.0 0.0 0.2" rpy="0.0 0.0 0.0"/>
+        <origin xyz="0.0 0.0 0.0" rpy="0.0 0.0 0.0"/>
         <parent link="world"/>
         <child link="chassis"/>
     </joint>
-    <link name='chassis'>
+        <!-- Chassis, caja de control /-->
+    <link name="chassis">
         <inertial>
             <mass value="4"/>
-            <origin xyz="0 0 0" rpy=" 0 0 0"/>
+            <origin xyz="0.2990 0.1954 0.2118" rpy=" 0 0 0"/>
             <inertia
-            ixx="0.0001" ixy="0" ixz="0"
-            iyy="0.0001" iyz="0"
-            izz="0.0001"
+                ixx="0.0001" ixy="0" ixz="0"
+                iyy="0.0001" iyz="0"
+                izz="0.0001"
             />
         </inertial>
-        <collision name='collision'>
-            <origin xyz="0 0 0" rpy=" 0 0 0"/>
+        <collision name='chassis_collision'>
+            <origin xyz="0.299 0.1954 0.2118" rpy=" 0 0 0"/>
             <geometry>
-                <box size="0.200 0.200 0.100"/>
+            <box size="0.2000 0.2000 0.1000"/>
             </geometry>
         </collision>
         <visual name='chassis_visual'>
-            <origin xyz="0 0 0" rpy=" 0 0 0"/>
+            <origin xyz="0.299 0.1954 0.2118" rpy=" 0 0 0"/>
             <geometry>
-                <box size="0.200 0.200 0.100"/>
+            <box size="0.2000 0.200 0.1000"/>
             </geometry>
-            <material name="orange">
-                <color rgba="0 0.5 0.5 1"/>
-            </material>
         </visual>
     </link>
     <joint name="joint_1" type="revolute">
-        <origin xyz="-0.12 0.0 0.0" rpy="0.0 0.0 0.0"/>
+        <origin xyz="0.0 0.0 0.0" rpy="0.0 0.0 0.0"/>
         <parent link="chassis"/>
-        <child link="left_leg_rocker"/>
-        <axis xyz="0.0 1 0.0"/>
-        <limit lower="0.0" upper="0.0" effort="0.0" velocity="0.0"/>
+        <child link="right_leg_rocker"/>
+        <axis xyz="0.0 1.0 0.0"/>
+        <limit lower="0.0" upper="1.0" effort="1.0" velocity="1.0"/>
     </joint>
-    <link name="left_leg_rocker">
+    <link name="right_leg_rocker">
         <inertial>
-            <mass value="1"/>
-            <origin xyz="0 0 0" rpy=" 0 0 0"/>
-            <inertia
-            ixx="0.0001" ixy="0" ixz="0"
-            iyy="0.0001" iyz="0"
-            izz="0.0001"
-            />
+            <origin xyz="0.0 0.0 0.0" rpy="0.0 0.0 0.0"/>
+            <mass value="1.0"/>
+            <inertia ixx="0.0" ixy="0.0" ixz="0.0" iyy="0.0" iyz="0.0" izz="0.0"/>
         </inertial>
-        <visual name="left_leg_rocker_1">
+        <visual name="">
             <origin xyz="0.0 0.0 0.0" rpy="0.0 0.0 0.0"/>
             <geometry>
-                <box size="0.219 0.025 0.025"/>
+                <box size="0.0 0.0 0.0"/>
             </geometry>
             <material name="">
                 <color rgba="1.0 0.0 0.0 1.0"/>
+                <texture filename=""/>
             </material>
         </visual>
-        <collision name="left_leg_rocker_1">
+        <collision>
             <origin xyz="0.0 0.0 0.0" rpy="0.0 0.0 0.0"/>
             <geometry>
-                <box size="0.219 0.025 0.025"/>
-            </geometry>
-        </collision>
-        <visual name="left_leg_rocker_2">
-            <origin xyz="-0.00 0.0 0.05" rpy="0.0 0.78 0.0"/>
-            <geometry>
-                <box size="0.219 0.025 0.025"/>
-            </geometry>
-            <material name="">
-                <color rgba="1.0 0.0 0.0 1.0"/>
-            </material>
-        </visual>
-        <collision name="left_leg_rocker_2">
-            <origin xyz="-0.01 0.0 0.05" rpy="0.0 0.78 0.0"/>
-            <geometry>
-                <box size="0.219 0.025 0.025"/>
-            </geometry>
-        </collision>
-        <visual name="left_leg_rocker_3">
-            <origin xyz="0.01 0.0 0.025" rpy="0.0 -0.78 0.0"/>
-            <geometry>
-                <box size="0.056 0.025 0.025"/>
-            </geometry>
-            <material name="">
-                <color rgba="1.0 0.0 0.0 1.0"/>
-            </material>
-        </visual>
-        <collision name="left_leg_rocker_3">
-            <origin xyz="0.01 0.0 0.025" rpy="0.0 -0.78 0.0"/>
-            <geometry>
-                <box size="0.056 0.025 0.025"/>
+                <box size="0.0 0.0 0.0"/>
             </geometry>
         </collision>
