Commit message: Updated most values on visual and collision, only joint and inertial left

File: src/mark1_description/urdf/mark1_complete.xacro (robot description, xacro)
@@ -11,5 +11,5 @@
   <!-- Chassis, caja de control /-->
   <link name="chassis">
-      <pose>0.299 0.1954 0.2118 0 0 0</pose >
+      <!-- pose>0.299 0.1954 0.2118 0 0 0</pose/-->
     <!-- estos valores no se si sirve/-->
       <inertial>
@@ -17,7 +17,7 @@
         <origin xyz="0.2990 0.1954 0.2118" rpy=" 0 0 0"/>
         <inertia
-            ixx="0.0001" ixy="0" ixz="0"
-            iyy="0.0001" iyz="0"
-            izz="0.0001"
+            ixx="0.05" ixy="0" ixz="0"
+            iyy="0.05" iyz="0"
+            izz="0.05"
         />
       </inertial>
@@ -36,5 +36,5 @@
   </link>
   <joint name="joint_1" type="revolute">
-    <origin xyz="0.0 0.0 0.0" rpy="0.0 0.0 0.0"/>
+    <origin xyz="0.30859 0.0827 0.21179" rpy="0.0 0.0 0.0"/>
     <parent link="chassis"/>
     <child link="right_leg_rocker"/>
@@ -50,5 +50,5 @@
         <box size="0.2195 0.00254 0.00254"/>
       </geometry>
-      <origin rpy="0 0 0" xyz="0.30859 0.0827 0.021179"/>
+      <origin rpy="0 0 0" xyz="0.30859 0.0827 0.21179"/>
     </visual>
     <visual name="r_down_part_visual">
@@ -75,15 +75,24 @@
         <box size="0.225 0.00254 0.00254"/>
       </geometry>
-      <origin rpy="0 -0.78 0" xyz="0.11954 0.0827 0.0825"/>
+      <origin rpy="0 -0.78 0" xyz="0.119 0.0827 0.0825"/>
     </collision>
     <collision name="r_front_part_collision">
       <geometry>
-        <box size="56 25.4 25.4"/>
-      </geometry>
-      <origin rpy="0 0.78 0" xyz="437.89 82.7 179.3"/>
-    </collision>
+        <box size="0.056 0.00254 0.00254"/>
+      </geometry>
+      <origin rpy="0 0.78 0" xyz="0.43789 0.0827 0.1793"/>
+    </collision>
+    <inertial>
+      <mass value="1"/>
+      <origin xyz="0.2990 0.1954 0.2118" rpy=" 0 0 0"/>
+      <inertia
+          ixx="0.001" ixy="0" ixz="0"
+          iyy="0.001" iyz="0"
+          izz="0.001"
+      />
+    </inertial>
   </link>
   <joint name="joint_2" type="revolute">
-    <origin xyz="0.0 0.0 0.0" rpy="0.0 0.0 0.0"/>
+    <origin xyz="0.30859 0.3481 0.21179" rpy="0.0 0.0 0.0"/>
     <parent link="chassis"/>
     <child link="left_leg_rocker"/>
@@ -101,13 +110,13 @@
     <visual name="l_down_part_visual">
       <geometry>
-        <box size="0.2195 0.00254 0.00254"/>
-      </geometry>
-      <origin rpy="0 -0.78 0" xyz="0.30859 0.3481 0.21179"/>
+        <box size="0.225 0.00254 0.00254"/>
+      </geometry>
+      <origin rpy="0 -0.78 0" xyz="0.119 0.3481 0.0825"/>
     </visual>
     <visual name="l_front_part_visual">
       <geometry>
-        <box size="0.2195 0.00254 0.00254"/>
-      </geometry>
-      <origin rpy="0 -0.78 0" xyz="0.30859 0.3481 0.21179"/>
+        <box size="0.056 0.00254 0.00254"/>
+      </geometry>
+      <origin rpy="0 0.78 0" xyz="0.43789 0.3481 0.1793"/>
     </visual>
     <!-- collision	 /-->
@@ -120,17 +129,26 @@
     <collision name="l_down_part_collision">
       <geometry>
-        <box size="0.2195 0.00254 0.00254"/>
-      </geometry>
-      <origin rpy="0 -0.78 0" xyz="0.30859 0.3481 0.21179"/>
+        <box size="0.225 0.00254 0.00254"/>
+      </geometry>
+      <origin rpy="0 -0.78 0" xyz="0.119 0.3481 0.0825"/>
     </collision>
     <collision name="l_front_part_collision">
       <geometry>
-        <box size="0.2195 0.254 0.254"/>
-      </geometry>
-      <origin rpy="0 -0.78 0" xyz="0.30859 0.3481 0.21179"/>
-    </collision>
+        <box size="0.056 0.00254 0.00254"/>
+      </geometry>
+      <origin rpy="0 0.78 0" xyz="0.43789 0.3481 0.1793"/>
+    </collision>
+    <inertial>
+      <mass value="1"/>
+      <origin xyz="0.2990 0.1954 0.2118" rpy=" 0 0 0"/>
+      <inertia
+          ixx="0.001" ixy="0" ixz="0"
+          iyy="0.001" iyz="0"
+          izz="0.001"
+      />
+    </inertial>
   </link>
   <joint name="joint_3" type="revolute">
-    <origin xyz="0.0 0.0 0.0" rpy="0.0 0.0 0.0"/>
+    <origin xyz="0.438 0.0827 0.1793" rpy="0.0 0.0 0.0"/>
     <parent link="right_leg_rocker"/>
     <child link="right_leg_boogie"/>
@@ -149,5 +167,5 @@
     <visual name="r_front_visual">
       <geometry>
-        <box size="0.00254 0.1195 0.00254"/>
+        <box size="0.00254 0.00254 0.01195"/>
       </geometry>
       <origin rpy="0 0 0" xyz="0.4707 0.0827 0.09975"/>
@@ -155,5 +173,5 @@
     <visual name="r_back_visual">
       <geometry>
-        <box size="0.00254 0.1195 0.00254"/>
+        <box size="0.00254 0.00254 0.01195"/>
       </geometry>
       <origin rpy="0 0 0" xyz="0.4053 0.0827 0.09975"/>
@@ -162,5 +180,5 @@
     <collision name="r_base_collision">
       <geometry>
-        <box size="0.400 0.00254 0.00254"/>
+        <box size="0.0400 0.00254 0.00254"/>
       </geometry>
       <origin rpy="0 0 0" xyz="0.4380 0.0827 0.1722"/>
@@ -168,5 +186,5 @@
     <collision name="r_front_collision">
       <geometry>
-        <box size="0.00254 0.01195 0.00254"/>
+        <box size="0.00254 0.00254 0.01195"/>
       </geometry>
       <origin rpy="0 0 0" xyz="0.04707 0.0827 0.09975"/>
@@ -174,11 +192,20 @@
     <collision name="r_back_collision">
       <geometry>
-        <box size="0.00254 0.1195 0.00254"/>
+        <box size="0.00254 0.00254 0.01195"/>
       </geometry>
       <origin rpy="0 0 0" xyz="0.4053 0.0827 0.09975"/>
     </collision>
+    <inertial>
+      <mass value="1"/>
+      <origin xyz="0.2990 0.1954 0.2118" rpy=" 0 0 0"/>
+      <inertia
+          ixx="0.001" ixy="0" ixz="0"
+          iyy="0.001" iyz="0"
+          izz="0.001"
+      />
+    </inertial>
   </link>
   <joint name="joint_4" type="revolute">
-    <origin xyz="0.0 0.0 0.0" rpy="0.0 0.0 0.0"/>
+    <origin xyz="0.438 0.3481 0.1793" rpy="0.0 0.0 0.0"/>
     <parent link="left_leg_rocker"/>
     <child link="left_leg_boogie"/>
@@ -196,5 +223,5 @@
     <visual name="l_front_visual">
       <geometry>
-        <box size="0.00254 0.1195 0.00254"/>
+        <box size="0.00254 0.00254 0.01195"/>
       </geometry>
       <origin rpy="0 0 0" xyz="0.4707 0.3481 0.09975"/>
@@ -202,5 +229,5 @@
     <visual name="l_back_visual">
       <geometry>
-        <box size="0.00254 0.1195 0.00254"/>
+        <box size="0.00254 0.00254 0.01195"/>
       </geometry>
       <origin rpy="0 0 0" xyz="0.4053 0.3481 0.09975"/>
@@ -209,5 +236,5 @@
     <collision name="l_base_collision">
       <geometry>
-        <box size="0.400 0.00254 0.00254"/>
+        <box size="0.0400 0.00254 0.00254"/>
       </geometry>
       <origin rpy="0 0 0" xyz="0.4380 0.3481 0.1722"/>
@@ -215,5 +242,5 @@
     <collision name="l_front_collision">
       <geometry>
-        <box size="0.00254 0.1195 0.00254"/>
+        <box size="0.00254 0.00254 0.01195"/>
       </geometry>
       <origin rpy="0 0 0" xyz="0.4707 0.3481 0.09975"/>
@@ -221,11 +248,21 @@
     <collision name="l_back_collision">
       <geometry>
-        <box size="0.00254 0.1195 0.00254"/>
+        <box size="00.00254 0.00254 0.01195"/>
       </geometry>
       <origin rpy="0 0 0" xyz="0.4053 0.3481 0.09975"/>
     </collision>
-  </link>
+    <inertial>
+      <mass value="1"/>
+      <origin xyz="0.2990 0.1954 0.2118" rpy=" 0 0 0"/>
+      <inertia
+          ixx="0.0001" ixy="0" ixz="0"
+          iyy="0.0001" iyz="0"
+          izz="0.0001"
+      />
+    </inertial>
+  </link>
+ <!--Llantas, son 6 en total 3 a cada lado  ..................... /-->
   <joint name="joint_5" type="revolute">
-    <origin xyz="0.0 0.0 0.0" rpy="0.0 0.0 0.0"/>
+    <origin xyz="0.04 0.0025 0.04" rpy="0.0 0.0 0.0"/>
     <parent link="right_leg_boogie"/>
     <child link="right_wheel_front"/>
@@ -233,5 +270,4 @@
     <limit lower="0.0" upper="0.0" effort="0.0" velocity="0.0"/>
   </joint>
-  <!--Llantas, son 6 en total 3 a cada lado  ..................... /-->
   <!--Llantas derechas/-->
   <link name="right_wheel_front">
@@ -248,7 +284,16 @@
       </geometry>
     </collision>
+    <inertial>
+      <mass value="1"/>
+      <origin xyz="0.2990 0.1954 0.2118" rpy=" 0 0 0"/>
+      <inertia
+          ixx="0.0001" ixy="0" ixz="0"
+          iyy="0.0001" iyz="0"
+          izz="0.0001"
+      />
+    </inertial>
   </link>
   <joint name="joint_6" type="revolute">
-    <origin xyz="0.0 0.0 0.0" rpy="0.0 0.0 0.0"/>
+    <origin xyz="0.4180 0.00250 0.00400" rpy="0.0 0.0 0.0"/>
     <parent link="right_leg_boogie"/>
     <child link="right_wheel_medium"/>
@@ -269,7 +314,16 @@
       </geometry>
     </collision>
+    <inertial>
+      <mass value="1"/>
+      <origin xyz="0.2990 0.1954 0.2118" rpy=" 0 0 0"/>
+      <inertia
+          ixx="0.0001" ixy="0" ixz="0"
+          iyy="0.0001" iyz="0"
+          izz="0.0001"
+      />
+    </inertial>
   </link>
   <joint name="joint_7" type="revolute">
-    <origin xyz="0.0 0.0 0.0" rpy="0.0 0.0 0.0"/>
+    <origin xyz="0.4580 0.00250 0.00400" rpy="0.0 0.0 0.0"/>
     <parent link="right_leg_boogie"/>
     <child link="right_wheel_back"/>
@@ -290,7 +344,17 @@
       </geometry>
     </collision>
-  </link>
+    <inertial>
+      <mass value="1"/>
+      <origin xyz="0.2990 0.1954 0.2118" rpy=" 0 0 0"/>
+      <inertia
+          ixx="0.0001" ixy="0" ixz="0"
+          iyy="0.0001" iyz="0"
+          izz="0.0001"
+      />
+    </inertial>
+  </link>
+  <!--Llantas izquierdas/-->
   <joint name="joint_8" type="revolute">
-    <origin xyz="0.0 0.0 0.0" rpy="0.0 0.0 0.0"/>
+    <origin xyz="0.0040 0.4058 0.00400" rpy="0.0 0.0 0.0"/>
     <parent link="left_leg_boogie"/>
     <child link="left_wheel_front"/>
@@ -298,5 +362,4 @@
     <limit lower="0.0" upper="0.0" effort="0.0" velocity="0.0"/>
   </joint>
-  <!--Llantas izquierdas/-->
   <link name="left_wheel_front">
     <visual name="left_wheel_front_visual">
@@ -312,46 +375,12 @@
       </geometry>
     </collision>
-  </link>
-  <joint name="joint_9" type="revolute">
-    <origin xyz="0.0 0.0 0.0" rpy="0.0 0.0 0.0"/>
-    <parent link="left_leg_boogie"/>
-    <child link="left_wheel_medium"/>
-    <axis xyz="0.0 1.0 0.0"/>
-    <limit lower="0.0" upper="0.0" effort="0.0" velocity="0.0"/>
-  </joint>
-  <link name="left_wheel_medium">
-    <visual name="left_wheel_medium_visual">
-      <origin rpy="0 1.5707 1.5707" xyz="0.4180 0.4058 0.00400"/>
-      <geometry>
-        <cylinder length="0.00500" radius="0.00400"/>
-      </geometry>
-    </visual>
-    <collision name="left_wheel_medium_collision">
-      <origin rpy="0 1.5707 1.5707" xyz="0.4180 0.4058 0.00400"/>
-      <geometry>
-        <cylinder length="0.00500" radius="0.00400"/>
-      </geometry>
-    </collision>
-  </link>
-  <joint name="joint_10" type="revolute">
-    <origin xyz="0.0 0.0 0.0" rpy="0.0 0.0 0.0"/>
-    <parent link="left_leg_boogie"/>
-    <child link="left_wheel_back"/>
-    <axis xyz="0.0 1.0 0.0"/>
-    <limit lower="0.0" upper="0.0" effort="0.0" velocity="0.0"/>
-  </joint>
-  <link name="left_wheel_back">
-    <visual name="left_wheel_back_visual">
-      <origin rpy="0 1.5707 1.5707" xyz="0.4580 0.4058 0.00400"/>
-      <geometry>
-        <cylinder length="0.00500" radius="0.00400"/>
-      </geometry>
-    </visual>
-    <collision name="left_wheel_back_collision">
-      <origin rpy="0 1.5707 1.5707" xyz="0.4580 0.4058 0.00400"/>
-      <geometry>
-        <cylinder length="0.00500" radius="0.00400"/>
-      </geometry>
-    </collision>
+    <inertial>
+      <mass value="1"/>
+      <origin xyz="0.2990 0.1954 0.2118" rpy=" 0 0 0"/>
+      <inertia
+          ixx="0.0001" ixy="0" ixz="0"
+          iyy="0.0001" iyz="0"
+          izz="0.0001"/>
+    </inertial>
   </link>
 </robot>

Commit message: Completed Wheels

File: src/mark1_description/urdf/mark1_complete.xacro (robot description, xacro)
@@ -384,3 +384,62 @@
     </inertial>
   </link>
+  <joint name="joint_9" type="revolute">
+    <origin xyz="0.4180 0.4058 0.00400" rpy="0.0 0.0 0.0"/>
+    <parent link="left_leg_boogie"/>
+    <child link="left_wheel_medium"/>
+    <axis xyz="0.0 1.0 0.0"/>
+    <limit lower="0.0" upper="0.0" effort="0.0" velocity="0.0"/>
+  </joint>
+  <link name="left_wheel_medium">
+    <visual name="left_wheel_medium_visual">
+      <origin rpy="0 1.5707 1.5707" xyz="0.4180 0.4058 0.00400"/>
+      <geometry>
+        <cylinder length="0.00500" radius="0.00400"/>
+      </geometry>
+    </visual>
+    <collision name="left_wheel_medium_collision">
+      <origin rpy="0 1.5707 1.5707" xyz="0.4180 0.4058 0.00400"/>
+      <geometry>
+        <cylinder length="0.00500" radius="0.00400"/>
+      </geometry>
+    </collision>
+    <inertial>
+      <mass value="1"/>
+      <origin xyz="0.2990 0.1954 0.2118" rpy=" 0 0 0"/>
+      <inertia
+          ixx="0.0001" ixy="0" ixz="0"
+          iyy="0.0001" iyz="0"
+          izz="0.0001"
+      />
+    </inertial>
+  </link>
+  <joint name="joint_10" type="revolute">
+    <origin xyz="0.4580 0.4058 0.00400" rpy="0.0 0.0 0.0"/>
+    <parent link="left_leg_boogie"/>
+    <child link="left_wheel_back"/>
+    <axis xyz="0.0 1.0 0.0"/>
+    <limit lower="0.0" upper="0.0" effort="0.0" velocity="0.0"/>
+  </joint>
+  <link name="left_wheel_back">
+    <visual name="left_wheel_back_visual">
+      <origin rpy="0 1.5707 1.5707" xyz="0.4580 0.4058 0.00400"/>
+      <geometry>
+        <cylinder length="0.00500" radius="0.00400"/>
+      </geometry>
+    </visual>
+    <collision name="left_wheel_back_collision">
+      <origin rpy="0 1.5707 1.5707" xyz="0.4580 0.4058 0.00400"/>
+      <geometry>
+        <cylinder length="0.00500" radius="0.00400"/>
+      </geometry>
+    </collision>
+    <inertial>
+      <mass value="1"/>
+      <origin xyz="0.2990 0.1954 0.2118" rpy=" 0 0 0"/>
+      <inertia
+          ixx="0.0001" ixy="0" ixz="0"
+          iyy="0.0001" iyz="0"
+          izz="0.0001"/>
+    </inertial>
+  </link>
 </robot>
