Commit message: Mark2

File: src/mark1_description/urdf/mark2.xacro (robot description, xacro)
@@ -1,23 +1,24 @@
 <?xml version='1.0'?>
 <robot name="mark2" xmlns:xacro="http://www.ros.org/wiki/xacro">
+    <!--
     <link name="world"></link>
     <joint name="joint_n" type="fixed">
-        <origin xyz="0.0 0.0 0.0" rpy="0.0 0.0 0.0"/>
+        <origin xyz="0.0 0.0 0.16" rpy="0.0 0.0 0.0"/>
         <parent link="world"/>
         <child link="chassis"/>
     </joint>
-        <!-- Chassis, caja de control /-->
+    -->
     <link name="chassis">
         <inertial>
-            <mass value="4"/>
-            <origin xyz="0.2990 0.1954 0.2118" rpy=" 0 0 0"/>
-            <inertia
-                ixx="0.0001" ixy="0" ixz="0"
-                iyy="0.0001" iyz="0"
-                izz="0.0001"
+            <mass value="3"/>
+            <origin xyz="0.0 0.0 0.0" rpy=" 0 0 0"/>
+            <inertia
+                ixx="0.05" ixy="0" ixz="0"
+                iyy="0.05" iyz="0"
+                izz="0.05"
             />
         </inertial>
         <collision name='chassis_collision'>
-            <origin xyz="0.299 0.1954 0.2118" rpy=" 0 0 0"/>
+            <origin xyz="0.0 0.0 0.0" rpy=" 0 0 0"/>
             <geometry>
             <box size="0.2000 0.2000 0.1000"/>
@@ -25,5 +26,5 @@
         </collision>
         <visual name='chassis_visual'>
-            <origin xyz="0.299 0.1954 0.2118" rpy=" 0 0 0"/>
+            <origin xyz="0.0 0.0 0.0" rpy=" 0 0 0"/>
             <geometry>
             <box size="0.2000 0.200 0.1000"/>
@@ -32,32 +33,406 @@
     </link>
     <joint name="joint_1" type="revolute">
-        <origin xyz="0.0 0.0 0.0" rpy="0.0 0.0 0.0"/>
+        <origin xyz="0.0 -0.1012 0.0" rpy="0.0 0.0 0.0"/>
         <parent link="chassis"/>
         <child link="right_leg_rocker"/>
         <axis xyz="0.0 1.0 0.0"/>
-        <limit lower="0.0" upper="1.0" effort="1.0" velocity="1.0"/>
+        <limit lower="-1.0" upper="1.0" effort="1.0" velocity="1.0"/>
     </joint>
     <link name="right_leg_rocker">
-        <inertial>
-            <origin xyz="0.0 0.0 0.0" rpy="0.0 0.0 0.0"/>
-            <mass value="1.0"/>
-            <inertia ixx="0.0" ixy="0.0" ixz="0.0" iyy="0.0" iyz="0.0" izz="0.0"/>
-        </inertial>
-        <visual name="">
-            <origin xyz="0.0 0.0 0.0" rpy="0.0 0.0 0.0"/>
-            <geometry>
-                <box size="0.0 0.0 0.0"/>
-            </geometry>
-            <material name="">
-                <color rgba="1.0 0.0 0.0 1.0"/>
-                <texture filename=""/>
-            </material>
-        </visual>
-        <collision>
-            <origin xyz="0.0 0.0 0.0" rpy="0.0 0.0 0.0"/>
-            <geometry>
-                <box size="0.0 0.0 0.0"/>
-            </geometry>
-        </collision>
+        <!-- visual /-->
+        <visual name="r_up_part_visual">
+            <geometry>
+                <box size="0.2195 0.00254 0.00254"/>
+            </geometry>
+            <origin rpy="0 0 0" xyz="0.0 0.0 0.0"/>
+        </visual>
+        <visual name="r_down_part_visual">
+            <geometry>
+                <box size="0.173 0.00254 0.00254"/>
+            </geometry>
+            <origin rpy="0 -1.1659 0" xyz="-0.1436 0.0 -0.0807"/>
+        </visual>
+        <visual name="r_front_part_visual">
+            <geometry>
+                <box size="0.09741 0.00254 0.00254"/>
+            </geometry>
+            <origin rpy="0 1.1522 0" xyz="0.1295 0.0 -0.0445"/>
+        </visual>
+        <!-- collision /-->
+        <collision name="r_up_part_collision">
+            <geometry>
+                <box size="0.2195 0.00254 0.00254"/>
+            </geometry>
+            <origin rpy="0 0 0" xyz="0.0 0.0 0.0"/>
+        </collision>
+        <collision name="r_down_part_collision">
+            <geometry>
+                <box size="0.173 0.00254 0.00254"/>
+            </geometry>
+            <origin rpy="0 -1.1659 0" xyz="-0.1436 0.0 -0.0807"/>
+        </collision>
+        <collision name="r_front_part_collision">
+            <geometry>
+                <box size="0.09741 0.00254 0.00254"/>
+            </geometry>
+            <origin rpy="0 1.1522 0" xyz="0.1295 0.0 -0.0445"/>
+        </collision>
+        <inertial>
+            <mass value="1"/>
+            <origin xyz="0.0 0.0 0.0" rpy=" 0 0 0"/>
+            <inertia
+                ixx="0.001" ixy="0" ixz="0"
+                iyy="0.001" iyz="0"
+                izz="0.001"
+            />
+        </inertial>
+    </link>
+    <joint name="joint_2" type="revolute">
+        <origin xyz="0.0 0.1012 0.0" rpy="0.0 0.0 0.0"/>
+        <parent link="chassis"/>
+        <child link="left_leg_rocker"/>
+        <axis xyz="0.0 1.0 0.0"/>
+        <limit lower="-1.0" upper="1.0" effort="1.0" velocity="1.0"/>
+    </joint>
+    <link name="left_leg_rocker">
+        <!-- visual /-->
+        <visual name="l_up_part_visual">
+            <geometry>
+                <box size="0.2195 0.00254 0.00254"/>
+            </geometry>
+            <origin rpy="0 0 0" xyz="0.0 0.0 0.0"/>
+        </visual>
+        <visual name="l_down_part_visual">
+            <geometry>
+                <box size="0.173 0.00254 0.00254"/>
+            </geometry>
+            <origin rpy="0 -1.1659 0" xyz="-0.1436 0.0 -0.0807"/>
+        </visual>
+        <visual name="l_front_part_visual">
+            <geometry>
+                <box size="0.09741 0.00254 0.00254"/>
+            </geometry>
+            <origin rpy="0 1.1522 0" xyz="0.1295 0.0 -0.0445"/>
+        </visual>
+        <!-- collision /-->
+        <collision name="l_up_part_collision">
+            <geometry>
+                <box size="0.2195 0.00254 0.00254"/>
+            </geometry>
+            <origin rpy="0 0 0" xyz="0.0 0.0 0.0"/>
+        </collision>
+        <collision name="l_down_part_collision">
+            <geometry>
+                <box size="0.173 0.00254 0.00254"/>
+            </geometry>
+            <origin rpy="0 -1.1659 0" xyz="-0.1436 0.0 -0.0807"/>
+        </collision>
+        <collision name="l_front_part_collision">
+            <geometry>
+                <box size="0.09741 0.00254 0.00254"/>
+            </geometry>
+            <origin rpy="0 1.1522 0" xyz="0.1295 0.0 -0.0445"/>
+        </collision>
+        <inertial>
+            <mass value="1"/>
+            <origin xyz="0.0 0.0 0.0" rpy=" 0 0 0"/>
+            <inertia
+                ixx="0.001" ixy="0" ixz="0"
+                iyy="0.001" iyz="0"
+                izz="0.001"
+            />
+        </inertial>
+    </link>
+    <joint name="joint_3" type="revolute">
+        <origin rpy="0 0 0" xyz="0.1493 0.0 -0.089"/>
+        <parent link="right_leg_rocker"/>
+        <child link="right_leg_boogie"/>
+        <axis xyz="0.0 1.0 0.0"/>
+        <limit lower="-1.0" upper="1.0" effort="1.0" velocity="1.0"/>
+    </joint>
+    <link name="right_leg_boogie">
+        <!-- visual /-->
+        <visual name="r_base_visual">
+            <geometry>
+                <box size="0.200 0.00254 0.00254"/>
+            </geometry>
+            <origin rpy="0 0 0" xyz="0.0 0.0 0.0"/>
+        </visual>
+        <visual name="r_front_visual">
+            <geometry>
+                <box size="0.00254 0.00254 0.0695"/>
+            </geometry>
+            <origin rpy="0 0 0" xyz="0.1 0.0 -0.03475"/>
+        </visual>
+        <visual name="r_back_visual">
+            <geometry>
+                <box size="0.00254 0.00254 0.0695"/>
+            </geometry>
+            <origin rpy="0 0 0" xyz="-0.1 0.0 -0.03475"/>
+        </visual>
+        <!-- collision /-->
+        <collision name="r_base_collision">
+            <geometry>
+                <box size="0.200 0.00254 0.00254"/>
+            </geometry>
+            <origin rpy="0 0 0" xyz="0.0 0.0 0.0"/>
+        </collision>
+        <collision name="r_front_collision">
+            <geometry>
+                <box size="0.00254 0.00254 0.0695"/>
+            </geometry>
+            <origin rpy="0 0 0" xyz="0.1 0.0 -0.03475"/>
+        </collision>
+        <collision name="r_back_collision">
+            <geometry>
+                <box size="0.00254 0.00254 0.0695"/>
+            </geometry>
+            <origin rpy="0 0 0" xyz="-0.1 0.0 -0.03475"/>
+        </collision>
+        <inertial>
+        <mass value="0.001"/>
+        <origin rpy="0 0 0" xyz="0.0 0.0 0.0"/>
+        <inertia
+            ixx="0.001" ixy="0" ixz="0"
+            iyy="0.001" iyz="0"
+            izz="0.001"
+        />
+        </inertial>
+    </link>
+    <joint name="joint_4" type="revolute">
+        <origin rpy="0 0 0" xyz="0.1493 0.0 -0.089"/>
+        <parent link="left_leg_rocker"/>
+        <child link="left_leg_boogie"/>
+        <axis xyz="0.0 1.0 0.0"/>
+        <limit lower="-1.0" upper="1.0" effort="1.0" velocity="1.0"/>
+    </joint>
+    <link name="left_leg_boogie">
+        <!-- visual /-->
+        <visual name="l_base_visual">
+            <geometry>
+                <box size="0.200 0.00254 0.00254"/>
+            </geometry>
+            <origin rpy="0 0 0" xyz="0.0 0.0 0.0"/>
+        </visual>
+        <visual name="l_front_visual">
+            <geometry>
+                <box size="0.00254 0.00254 0.0695"/>
+            </geometry>
+            <origin rpy="0 0 0" xyz="0.1 0.0 -0.03475"/>
+        </visual>
+        <visual name="l_back_visual">
+            <geometry>
+                <box size="0.00254 0.00254 0.0695"/>
+            </geometry>
+            <origin rpy="0 0 0" xyz="-0.1 0.0 -0.03475"/>
+        </visual>
+        <!-- collision /-->
+        <collision name="l_base_collision">
+            <geometry>
+                <box size="0.200 0.00254 0.00254"/>
+            </geometry>
+            <origin rpy="0 0 0" xyz="0.0 0.0 0.0"/>
+        </collision>
+        <collision name="l_front_collision">
+            <geometry>
+                <box size="0.00254 0.00254 0.0695"/>
+            </geometry>
+            <origin rpy="0 0 0" xyz="0.1 0.0 -0.03475"/>
+        </collision>
+        <collision name="l_back_collision">
+            <geometry>
+                <box size="0.00254 0.00254 0.0695"/>
+            </geometry>
+            <origin rpy="0 0 0" xyz="-0.1 0.0 -0.03475"/>
+        </collision>
+        <inertial>
+        <mass value="0.001"/>
+        <origin rpy="0 0 0" xyz="0.0 0.0 0.0"/>
+        <inertia
+            ixx="0.001" ixy="0" ixz="0"
+            iyy="0.001" iyz="0"
+            izz="0.001"
+        />
+        </inertial>
+    </link>
+    <joint name="joint_5" type="revolute">
+        <origin xyz="0.1 0.0 -0.0695" rpy="0.0 1.5707 0.0"/>
+        <parent link="right_leg_boogie"/>
+        <child link="right_wheel_front"/>
+        <axis xyz="0.0 1.0 0.0"/>
+        <limit lower="-3.14" upper="3.14" effort="1.0" velocity="1.0"/>
+    </joint>
+    <link name="right_wheel_front">
+        <visual name="right_wheel_front_visual">
+            <origin rpy="1.5707 0.0 0.0" xyz="0.0 0.0 0.0"/>
+            <geometry>
+                <cylinder length="0.00500" radius="0.00400"/>
+            </geometry>
+        </visual>
+        <collision name="right_wheel_front_collision">
+            <origin rpy="1.5707 0.0 0.0" xyz="0.0 0.0 0.0"/>
+            <geometry>
+                <cylinder length="0.00500" radius="0.00400"/>
+            </geometry>
+        </collision>
+        <inertial>
+            <mass value="0.0001"/>
+            <origin xyz="0.2990 0.1954 0.2118" rpy=" 0 0 0"/>
+            <inertia
+                ixx="0.0001" ixy="0" ixz="0"
+                iyy="0.0001" iyz="0"
+                izz="0.0001"
+            />
+        </inertial>
+    </link>
+    <joint name="joint_6" type="revolute">
+        <origin xyz="-0.1 0.0 -0.0695" rpy="0.0 1.5707 0.0"/>
+        <parent link="right_leg_boogie"/>
+        <child link="right_wheel_medium"/>
+        <axis xyz="0.0 1.0 0.0"/>
+        <limit lower="-3.14" upper="3.14" effort="1.0" velocity="1.0"/>
+    </joint>
+    <link name="right_wheel_medium">
+        <visual name="right_wheel_front_visual">
+            <origin rpy="1.5707 0.0 0.0" xyz="0.0 0.0 0.0"/>
+            <geometry>
+                <cylinder length="0.00500" radius="0.00400"/>
+            </geometry>
+        </visual>
+        <collision name="right_wheel_front_collision">
+            <origin rpy="1.5707 0.0 0.0" xyz="0.0 0.0 0.0"/>
+            <geometry>
+                <cylinder length="0.00500" radius="0.00400"/>
+            </geometry>
+        </collision>
+        <inertial>
+            <mass value="0.0001"/>
+            <origin xyz="0.2990 0.1954 0.2118" rpy=" 0 0 0"/>
+            <inertia
+                ixx="0.0001" ixy="0" ixz="0"
+                iyy="0.0001" iyz="0"
+                izz="0.0001"
+            />
+        </inertial>
+    </link>
+    <joint name="joint_7" type="revolute">
+        <origin xyz="-0.1776 0.0 -0.1586" rpy="0.0 1.5707 0.0"/>
+        <parent link="right_leg_rocker"/>
+        <child link="right_wheel_back"/>
+        <axis xyz="0.0 1.0 0.0"/>
+        <limit lower="-3.14" upper="3.14" effort="1.0" velocity="1.0"/>
+    </joint>
+    <link name="right_wheel_back">
+        <visual name="right_wheel_front_visual">
+            <origin rpy="1.5707 0.0 0.0" xyz="0.0 0.0 0.0"/>
+            <geometry>
+                <cylinder length="0.00500" radius="0.00400"/>
+            </geometry>
+        </visual>
+        <collision name="right_wheel_front_collision">
+            <origin rpy="1.5707 0.0 0.0" xyz="0.0 0.0 0.0"/>
+            <geometry>
+                <cylinder length="0.00500" radius="0.00400"/>
+            </geometry>
+        </collision>
+        <inertial>
+            <mass value="0.0001"/>
+            <origin xyz="0.2990 0.1954 0.2118" rpy=" 0 0 0"/>
+            <inertia
+                ixx="0.0001" ixy="0" ixz="0"
+                iyy="0.0001" iyz="0"
+                izz="0.0001"
+            />
+        </inertial>
+    </link>
+    <joint name="joint_8" type="revolute">
+        <origin xyz="0.1 0.0 -0.0695" rpy="0.0 1.5707 0.0"/>
+        <parent link="left_leg_boogie"/>
+        <child link="left_wheel_front"/>
+        <axis xyz="0.0 1.0 0.0"/>
+        <limit lower="-3.14" upper="3.14" effort="1.0" velocity="1.0"/>
+    </joint>
+    <link name="left_wheel_front">
+        <visual name="left_wheel_front_visual">
+            <origin rpy="1.5707 0.0 0.0" xyz="0.0 0.0 0.0"/>
+            <geometry>
+                <cylinder length="0.00500" radius="0.00400"/>
+            </geometry>
+        </visual>
+        <collision name="left_wheel_front_collision">
+            <origin rpy="1.5707 0.0 0.0" xyz="0.0 0.0 0.0"/>
+            <geometry>
+                <cylinder length="0.00500" radius="0.00400"/>
+            </geometry>
+        </collision>
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