Commit message: Mark(2)

File: src/mark1_description/urdf/mark2.xacro (robot description, xacro)
@@ -4,5 +4,5 @@
     <link name="world"></link>
     <joint name="joint_n" type="fixed">
-        <origin xyz="0.0 0.0 0.16" rpy="0.0 0.0 0.0"/>
+        <origin xyz="0.0 0.0 0.2" rpy="0.0 0.0 0.0"/>
         <parent link="world"/>
         <child link="chassis"/>
@@ -28,5 +28,5 @@
             <origin xyz="0.0 0.0 0.0" rpy=" 0 0 0"/>
             <geometry>
-            <box size="0.2000 0.200 0.1000"/>
+            <box size="0.2000 0.2000 0.1000"/>
             </geometry>
         </visual>
@@ -43,5 +43,5 @@
         <visual name="r_up_part_visual">
             <geometry>
-                <box size="0.2195 0.00254 0.00254"/>
+                <box size="0.2195 0.0254 0.0254"/>
             </geometry>
             <origin rpy="0 0 0" xyz="0.0 0.0 0.0"/>
@@ -49,5 +49,5 @@
         <visual name="r_down_part_visual">
             <geometry>
-                <box size="0.173 0.00254 0.00254"/>
+                <box size="0.173 0.0254 0.0254"/>
             </geometry>
             <origin rpy="0 -1.1659 0" xyz="-0.1436 0.0 -0.0807"/>
@@ -55,5 +55,5 @@
         <visual name="r_front_part_visual">
             <geometry>
-                <box size="0.09741 0.00254 0.00254"/>
+                <box size="0.09741 0.0254 0.0254"/>
             </geometry>
             <origin rpy="0 1.1522 0" xyz="0.1295 0.0 -0.0445"/>
@@ -62,5 +62,5 @@
         <collision name="r_up_part_collision">
             <geometry>
-                <box size="0.2195 0.00254 0.00254"/>
+                <box size="0.2195 0.0254 0.0254"/>
             </geometry>
             <origin rpy="0 0 0" xyz="0.0 0.0 0.0"/>
@@ -68,5 +68,5 @@
         <collision name="r_down_part_collision">
             <geometry>
-                <box size="0.173 0.00254 0.00254"/>
+                <box size="0.173 0.0254 0.0254"/>
             </geometry>
             <origin rpy="0 -1.1659 0" xyz="-0.1436 0.0 -0.0807"/>
@@ -74,5 +74,5 @@
         <collision name="r_front_part_collision">
             <geometry>
-                <box size="0.09741 0.00254 0.00254"/>
+                <box size="0.09741 0.0254 0.0254"/>
             </geometry>
             <origin rpy="0 1.1522 0" xyz="0.1295 0.0 -0.0445"/>
@@ -99,5 +99,5 @@
         <visual name="l_up_part_visual">
             <geometry>
-                <box size="0.2195 0.00254 0.00254"/>
+                <box size="0.2195 0.0254 0.0254"/>
             </geometry>
             <origin rpy="0 0 0" xyz="0.0 0.0 0.0"/>
@@ -105,5 +105,5 @@
         <visual name="l_down_part_visual">
             <geometry>
-                <box size="0.173 0.00254 0.00254"/>
+                <box size="0.173 0.0254 0.0254"/>
             </geometry>
             <origin rpy="0 -1.1659 0" xyz="-0.1436 0.0 -0.0807"/>
@@ -111,5 +111,5 @@
         <visual name="l_front_part_visual">
             <geometry>
-                <box size="0.09741 0.00254 0.00254"/>
+                <box size="0.09741 0.0254 0.0254"/>
             </geometry>
             <origin rpy="0 1.1522 0" xyz="0.1295 0.0 -0.0445"/>
@@ -118,5 +118,5 @@
         <collision name="l_up_part_collision">
             <geometry>
-                <box size="0.2195 0.00254 0.00254"/>
+                <box size="0.2195 0.0254 0.0254"/>
             </geometry>
             <origin rpy="0 0 0" xyz="0.0 0.0 0.0"/>
@@ -124,5 +124,5 @@
         <collision name="l_down_part_collision">
             <geometry>
-                <box size="0.173 0.00254 0.00254"/>
+                <box size="0.173 0.0254 0.0254"/>
             </geometry>
             <origin rpy="0 -1.1659 0" xyz="-0.1436 0.0 -0.0807"/>
@@ -130,5 +130,5 @@
         <collision name="l_front_part_collision">
             <geometry>
-                <box size="0.09741 0.00254 0.00254"/>
+                <box size="0.09741 0.0254 0.0254"/>
             </geometry>
             <origin rpy="0 1.1522 0" xyz="0.1295 0.0 -0.0445"/>
@@ -155,5 +155,5 @@
         <visual name="r_base_visual">
             <geometry>
-                <box size="0.200 0.00254 0.00254"/>
+                <box size="0.200 0.0254 0.0254"/>
             </geometry>
             <origin rpy="0 0 0" xyz="0.0 0.0 0.0"/>
@@ -161,5 +161,5 @@
         <visual name="r_front_visual">
             <geometry>
-                <box size="0.00254 0.00254 0.0695"/>
+                <box size="0.0254 0.0254 0.0695"/>
             </geometry>
             <origin rpy="0 0 0" xyz="0.1 0.0 -0.03475"/>
@@ -167,5 +167,5 @@
         <visual name="r_back_visual">
             <geometry>
-                <box size="0.00254 0.00254 0.0695"/>
+                <box size="0.0254 0.0254 0.0695"/>
             </geometry>
             <origin rpy="0 0 0" xyz="-0.1 0.0 -0.03475"/>
@@ -211,5 +211,5 @@
         <visual name="l_base_visual">
             <geometry>
-                <box size="0.200 0.00254 0.00254"/>
+                <box size="0.200 0.0254 0.0254"/>
             </geometry>
             <origin rpy="0 0 0" xyz="0.0 0.0 0.0"/>
@@ -217,5 +217,5 @@
         <visual name="l_front_visual">
             <geometry>
-                <box size="0.00254 0.00254 0.0695"/>
+                <box size="0.0254 0.0254 0.0695"/>
             </geometry>
             <origin rpy="0 0 0" xyz="0.1 0.0 -0.03475"/>
@@ -223,5 +223,5 @@
         <visual name="l_back_visual">
             <geometry>
-                <box size="0.00254 0.00254 0.0695"/>
+                <box size="0.0254 0.0254 0.0695"/>
             </geometry>
             <origin rpy="0 0 0" xyz="-0.1 0.0 -0.03475"/>
@@ -230,5 +230,5 @@
         <collision name="l_base_collision">
             <geometry>
-                <box size="0.200 0.00254 0.00254"/>
+                <box size="0.200 0.0254 0.0254"/>
             </geometry>
             <origin rpy="0 0 0" xyz="0.0 0.0 0.0"/>
@@ -236,5 +236,5 @@
         <collision name="l_front_collision">
             <geometry>
-                <box size="0.00254 0.00254 0.0695"/>
+                <box size="0.0254 0.0254 0.0695"/>
             </geometry>
             <origin rpy="0 0 0" xyz="0.1 0.0 -0.03475"/>
@@ -242,5 +242,5 @@
         <collision name="l_back_collision">
             <geometry>
-                <box size="0.00254 0.00254 0.0695"/>
+                <box size="0.0254 0.0254 0.0695"/>
             </geometry>
             <origin rpy="0 0 0" xyz="-0.1 0.0 -0.03475"/>
@@ -256,10 +256,10 @@
         </inertial>
     </link>
-    <joint name="joint_5" type="revolute">
-        <origin xyz="0.1 0.0 -0.0695" rpy="0.0 1.5707 0.0"/>
+    <joint name="joint_5" type="continuous">
+        <origin xyz="0.1 -0.0377 -0.0695" rpy="0.0 1.5707 0.0"/>
         <parent link="right_leg_boogie"/>
         <child link="right_wheel_front"/>
         <axis xyz="0.0 1.0 0.0"/>
-        <limit lower="-3.14" upper="3.14" effort="1.0" velocity="1.0"/>
+        <limit effort="1.0" velocity="4.0"/>
     </joint>
     <link name="right_wheel_front">
@@ -267,5 +267,5 @@
             <origin rpy="1.5707 0.0 0.0" xyz="0.0 0.0 0.0"/>
             <geometry>
-                <cylinder length="0.00500" radius="0.00400"/>
+                <cylinder length="0.0500" radius="0.0400"/>
             </geometry>
         </visual>
@@ -273,5 +273,5 @@
             <origin rpy="1.5707 0.0 0.0" xyz="0.0 0.0 0.0"/>
             <geometry>
-                <cylinder length="0.00500" radius="0.00400"/>
+                <cylinder length="0.0500" radius="0.0400"/>
             </geometry>
         </collision>
@@ -286,10 +286,10 @@
         </inertial>
     </link>
-    <joint name="joint_6" type="revolute">
-        <origin xyz="-0.1 0.0 -0.0695" rpy="0.0 1.5707 0.0"/>
+    <joint name="joint_6" type="continuous">
+        <origin xyz="-0.1 -0.0377 -0.0695" rpy="0.0 1.5707 0.0"/>
         <parent link="right_leg_boogie"/>
         <child link="right_wheel_medium"/>
         <axis xyz="0.0 1.0 0.0"/>
-        <limit lower="-3.14" upper="3.14" effort="1.0" velocity="1.0"/>
+        <limit effort="1.0" velocity="4.0"/>
     </joint>
     <link name="right_wheel_medium">
@@ -297,5 +297,5 @@
             <origin rpy="1.5707 0.0 0.0" xyz="0.0 0.0 0.0"/>
             <geometry>
-                <cylinder length="0.00500" radius="0.00400"/>
+                <cylinder length="0.0500" radius="0.0400"/>
             </geometry>
         </visual>
@@ -303,5 +303,5 @@
             <origin rpy="1.5707 0.0 0.0" xyz="0.0 0.0 0.0"/>
             <geometry>
-                <cylinder length="0.00500" radius="0.00400"/>
+                <cylinder length="0.0500" radius="0.0400"/>
             </geometry>
         </collision>
@@ -316,10 +316,10 @@
         </inertial>
     </link>
-    <joint name="joint_7" type="revolute">
-        <origin xyz="-0.1776 0.0 -0.1586" rpy="0.0 1.5707 0.0"/>
+    <joint name="joint_7" type="continuous">
+        <origin xyz="-0.1776 -0.0377 -0.1586" rpy="0.0 1.5707 0.0"/>
         <parent link="right_leg_rocker"/>
         <child link="right_wheel_back"/>
         <axis xyz="0.0 1.0 0.0"/>
-        <limit lower="-3.14" upper="3.14" effort="1.0" velocity="1.0"/>
+        <limit effort="1.0" velocity="4.0"/>
     </joint>
     <link name="right_wheel_back">
@@ -327,5 +327,5 @@
             <origin rpy="1.5707 0.0 0.0" xyz="0.0 0.0 0.0"/>
             <geometry>
-                <cylinder length="0.00500" radius="0.00400"/>
+                <cylinder length="0.0500" radius="0.0400"/>
             </geometry>
         </visual>
@@ -333,5 +333,5 @@
             <origin rpy="1.5707 0.0 0.0" xyz="0.0 0.0 0.0"/>
             <geometry>
-                <cylinder length="0.00500" radius="0.00400"/>
+                <cylinder length="0.0500" radius="0.0400"/>
             </geometry>
         </collision>
@@ -346,10 +346,10 @@
         </inertial>
     </link>
-    <joint name="joint_8" type="revolute">
-        <origin xyz="0.1 0.0 -0.0695" rpy="0.0 1.5707 0.0"/>
+    <joint name="joint_8" type="continuous">
+        <origin xyz="0.1 0.0377 -0.0695" rpy="0.0 1.5707 0.0"/>
         <parent link="left_leg_boogie"/>
         <child link="left_wheel_front"/>
         <axis xyz="0.0 1.0 0.0"/>
-        <limit lower="-3.14" upper="3.14" effort="1.0" velocity="1.0"/>
+        <limit effort="1.0" velocity="4.0"/>
     </joint>
     <link name="left_wheel_front">
@@ -357,5 +357,5 @@
             <origin rpy="1.5707 0.0 0.0" xyz="0.0 0.0 0.0"/>
             <geometry>
-                <cylinder length="0.00500" radius="0.00400"/>
+                <cylinder length="0.0500" radius="0.0400"/>
             </geometry>
         </visual>
@@ -363,5 +363,5 @@
             <origin rpy="1.5707 0.0 0.0" xyz="0.0 0.0 0.0"/>
             <geometry>
-                <cylinder length="0.00500" radius="0.00400"/>
+                <cylinder length="0.0500" radius="0.0400"/>
             </geometry>
         </collision>
@@ -376,10 +376,10 @@
         </inertial>
     </link>
-    <joint name="joint_9" type="revolute">
-        <origin xyz="-0.1 0.0 -0.0695" rpy="0.0 1.5707 0.0"/>
+    <joint name="joint_9" type="continuous">
+        <origin xyz="-0.1 0.0377 -0.0695" rpy="0.0 1.5707 0.0"/>
         <parent link="left_leg_boogie"/>
         <child link="left_wheel_medium"/>
         <axis xyz="0.0 1.0 0.0"/>
-        <limit lower="-3.14" upper="3.14" effort="1.0" velocity="1.0"/>
+        <limit effort="1.0" velocity="4.0"/>
     </joint>
     <link name="left_wheel_medium">
@@ -387,5 +387,5 @@
             <origin rpy="1.5707 0.0 0.0" xyz="0.0 0.0 0.0"/>
             <geometry>
-                <cylinder length="0.00500" radius="0.00400"/>
+                <cylinder length="0.0500" radius="0.0400"/>
             </geometry>
         </visual>
@@ -393,5 +393,5 @@
             <origin rpy="1.5707 0.0 0.0" xyz="0.0 0.0 0.0"/>
             <geometry>
-                <cylinder length="0.00500" radius="0.00400"/>
+                <cylinder length="0.0500" radius="0.0400"/>
             </geometry>
         </collision>
@@ -406,10 +406,10 @@
         </inertial>
     </link>
-    <joint name="joint_10" type="revolute">
-        <origin xyz="-0.1776 0.0 -0.1586" rpy="0.0 1.5707 0.0"/>
+    <joint name="joint_10" type="continuous">
+        <origin xyz="-0.1776 0.0377 -0.1586" rpy="0.0 1.5707 0.0"/>
         <parent link="left_leg_rocker"/>
         <child link="left_wheel_back"/>
         <axis xyz="0.0 1.0 0.0"/>
-        <limit lower="-3.14" upper="3.14" effort="1.0" velocity="1.0"/>
+        <limit effort="1.0" velocity="4.0"/>
     </joint>
     <link name="left_wheel_back">
@@ -417,5 +417,5 @@
             <origin rpy="1.5707 0.0 0.0" xyz="0.0 0.0 0.0"/>
             <geometry>
-                <cylinder length="0.00500" radius="0.00400"/>
+                <cylinder length="0.0500" radius="0.0400"/>
             </geometry>
         </visual>
@@ -423,5 +423,5 @@
             <origin rpy="1.5707 0.0 0.0" xyz="0.0 0.0 0.0"/>
             <geometry>
-                <cylinder length="0.00500" radius="0.00400"/>
+                <cylinder length="0.0500" radius="0.0400"/>
             </geometry>
         </collision>
@@ -436,3 +436,134 @@
         </inertial>
     </link>
+    <!-- differential -->
+    <joint name="joint_11" type="fixed">
+        <origin xyz="0.0 0.1012 0.08" rpy="0.0 0.0 0.0"/>
+        <parent link="right_leg_rocker"/>
+        <child link="diff"/>
+    </joint>
+    <link name="diff">
+        <visual name="">
+            <origin xyz="0.0 0.0 0.0" rpy="0.0 0.0 0.0"/>
+            <geometry>
+                <box size="0.01 0.22 0.01"/>
+            </geometry>
+        </visual>
+        <visual name="">
+            <origin xyz="0.0 0.105 -0.04" rpy="0.0 0.0 0.0"/>
+            <geometry>
+                <box size="0.01 0.01 0.08"/>
+            </geometry>
+        </visual>
+        <visual name="">
+            <origin xyz="0.0 -0.105 -0.04" rpy="0.0 0.0 0.0"/>
+            <geometry>
+                <box size="0.01 0.01 0.08"/>
+            </geometry>
+        </visual>
+        <collision>
+            <origin xyz="0.0 0.0 0.0" rpy="0.0 0.0 0.0"/>
+            <geometry>
+                <box size="0.01 0.22 0.01"/>
+            </geometry>
+        </collision>
+        <collision>
+            <origin xyz="0.0 0.105 -0.04" rpy="0.0 0.0 0.0"/>
+            <geometry>
+                <box size="0.01 0.01 0.08"/>
+            </geometry>
+        </collision>
+        <collision>
+            <origin xyz="0.0 -0.105 -0.04" rpy="0.0 0.0 0.0"/>
+            <geometry>
+                <box size="0.01 0.01 0.08"/>
+            </geometry>
+        </collision>
+        <inertial>
+            <origin xyz="0.0 0.0 0.0" rpy="0.0 0.0 0.0"/>
+            <mass value="0.001"/>
+            <inertia ixx="0.001" ixy="0.0" ixz="0.0" iyy="0.001" iyz="0.0" izz="0.001"/>
+        </inertial>
+    </link>
+    <!-- Transmission -->
+    <transmission name="tran1">
+        <type>transmission_interface/SimpleTransmission</type>
+        <joint name="joint_5">
+            <hardwareInterface>hardware_interface/VelocityJointInterface</hardwareInterface>
+        </joint>
+        <actuator name="Wheel_RF">
+            <mechanicalReduction>1</mechanicalReduction>
+        </actuator>
+    </transmission>
+    <transmission name="tran2">
+        <type>transmission_interface/SimpleTransmission</type>
+        <joint name="joint_6">
+            <hardwareInterface>hardware_interface/VelocityJointInterface</hardwareInterface>
+        </joint>
+        <actuator name="Wheel_RM">
+            <mechanicalReduction>1</mechanicalReduction>
+        </actuator>
+    </transmission>
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
Commit message: Mark2)

File: src/mark1_description/urdf/mark2.xacro (robot description, xacro)
@@ -1,20 +1,18 @@
 <?xml version='1.0'?>
 <robot name="mark2" xmlns:xacro="http://www.ros.org/wiki/xacro">
-    <!--
     <link name="world"></link>
-    <joint name="joint_n" type="fixed">
+    <joint name="joint_n" type="floating">
         <origin xyz="0.0 0.0 0.2" rpy="0.0 0.0 0.0"/>
         <parent link="world"/>
         <child link="chassis"/>
     </joint>
-    -->
     <link name="chassis">
         <inertial>
-            <mass value="3"/>
+            <mass value="1.5"/>
             <origin xyz="0.0 0.0 0.0" rpy=" 0 0 0"/>
             <inertia
-                ixx="0.05" ixy="0" ixz="0"
-                iyy="0.05" iyz="0"
-                izz="0.05"
+                ixx="0.00625" ixy="0" ixz="0"
+                iyy="0.00625" iyz="0"
+                izz="0.01"
             />
         </inertial>
@@ -174,5 +172,5 @@
         <collision name="r_base_collision">
             <geometry>
-                <box size="0.200 0.00254 0.00254"/>
+                <box size="0.200 0.0254 0.0254"/>
             </geometry>
             <origin rpy="0 0 0" xyz="0.0 0.0 0.0"/>
@@ -180,5 +178,5 @@
         <collision name="r_front_collision">
             <geometry>
-                <box size="0.00254 0.00254 0.0695"/>
+                <box size="0.0254 0.0254 0.0695"/>
             </geometry>
             <origin rpy="0 0 0" xyz="0.1 0.0 -0.03475"/>
@@ -186,10 +184,10 @@
         <collision name="r_back_collision">
             <geometry>
-                <box size="0.00254 0.00254 0.0695"/>
+                <box size="0.0254 0.0254 0.0695"/>
             </geometry>
             <origin rpy="0 0 0" xyz="-0.1 0.0 -0.03475"/>
         </collision>
         <inertial>
-        <mass value="0.001"/>
+        <mass value="0.01"/>
         <origin rpy="0 0 0" xyz="0.0 0.0 0.0"/>
         <inertia
@@ -247,5 +245,5 @@
         </collision>
         <inertial>
-        <mass value="0.001"/>
+        <mass value="0.01"/>
         <origin rpy="0 0 0" xyz="0.0 0.0 0.0"/>
         <inertia
@@ -261,5 +259,5 @@
         <child link="right_wheel_front"/>
         <axis xyz="0.0 1.0 0.0"/>
-        <limit effort="1.0" velocity="4.0"/>
+        <limit effort="100.0" velocity="4.0"/>
     </joint>
     <link name="right_wheel_front">
@@ -351,5 +349,5 @@
         <child link="left_wheel_front"/>
         <axis xyz="0.0 1.0 0.0"/>
-        <limit effort="1.0" velocity="4.0"/>
+        <limit effort="100.0" velocity="4.0"/>
     </joint>
     <link name="left_wheel_front">
@@ -547,5 +545,5 @@
     </gazebo>
     <gazebo reference="chassis">
-        <material>Gazebo/Red</material>
+        <material>Gazebo/Gray</material>
     </gazebo>
     <gazebo reference="right_wheel_front">
@@ -553,5 +551,5 @@
     </gazebo>
     <gazebo reference="right_wheel_medium">
-        <material>Gazebo/Black</material>
+        <material>Gazebo/Blue</material>
     </gazebo>
     <gazebo reference="right_wheel_back">
@@ -562,5 +560,5 @@
     </gazebo>
     <gazebo reference="left_wheel_medium">
-        <material>Gazebo/Black</material>
+        <material>Gazebo/Blue</material>
     </gazebo>
     <gazebo reference="left_wheel_back">
