Commit message: Control

File: src/mark1_description/urdf/mark2.xacro (robot description, xacro)
@@ -9,10 +9,10 @@
     <link name="chassis">
         <inertial>
-            <mass value="1.5"/>
+            <mass value="3.065"/>
             <origin xyz="0.0 0.0 0.0" rpy=" 0 0 0"/>
             <inertia
-                ixx="0.00625" ixy="0" ixz="0"
-                iyy="0.00625" iyz="0"
-                izz="0.01"
+                ixx="199.731" ixy="2.097" ixz="0.161"
+                iyy="182.087" iyz="0.079"
+                izz="267.088"
             />
         </inertial>
@@ -77,10 +77,10 @@
         </collision>
         <inertial>
-            <mass value="1"/>
+            <mass value="0.974"/>
             <origin xyz="0.0 0.0 0.0" rpy=" 0 0 0"/>
             <inertia
-                ixx="0.001" ixy="0" ixz="0"
-                iyy="0.001" iyz="0"
-                izz="0.001"
+                ixx="2555.119" ixy="60.204" ixz="-2683.738"
+                iyy="15204.978" iyz="16.365"
+                izz="12798.286"
             />
         </inertial>
@@ -133,10 +133,10 @@
         </collision>
         <inertial>
-            <mass value="1"/>
+            <mass value="0.974"/>
             <origin xyz="0.0 0.0 0.0" rpy=" 0 0 0"/>
             <inertia
-                ixx="0.001" ixy="0" ixz="0"
-                iyy="0.001" iyz="0"
-                izz="0.001"
+                ixx="2555.119" ixy="60.204" ixz="-2683.738"
+                iyy="15204.978" iyz="16.365"
+                izz="12798.286"
             />
         </inertial>
@@ -189,10 +189,10 @@
         </collision>
         <inertial>
-        <mass value="0.01"/>
+        <mass value="0.803"/>
         <origin rpy="0 0 0" xyz="0.0 0.0 0.0"/>
         <inertia
-            ixx="0.001" ixy="0" ixz="0"
-            iyy="0.001" iyz="0"
-            izz="0.001"
+            ixx="664.519" ixy="-9.047" ixz="224.365"
+                iyy="4936.122" iyz="26.955"
+                izz="4390.159"
         />
         </inertial>
@@ -245,11 +245,11 @@
         </collision>
         <inertial>
-        <mass value="0.01"/>
-        <origin rpy="0 0 0" xyz="0.0 0.0 0.0"/>
-        <inertia
-            ixx="0.001" ixy="0" ixz="0"
-            iyy="0.001" iyz="0"
-            izz="0.001"
-        />
+            <mass value="0.803"/>
+            <origin rpy="0 0 0" xyz="0.0 0.0 0.0"/>
+            <inertia
+                ixx="664.519" ixy="-9.047" ixz="224.365"
+                iyy="4936.122" iyz="26.955"
+                izz="4390.159"
+            />
         </inertial>
     </link>
@@ -259,5 +259,5 @@
         <child link="right_wheel_front"/>
         <axis xyz="0.0 1.0 0.0"/>
-        <limit effort="100.0" velocity="4.0"/>
+        <limit effort="100.0" velocity="15.0"/>
     </joint>
     <link name="right_wheel_front">
@@ -275,10 +275,10 @@
         </collision>
         <inertial>
-            <mass value="0.0001"/>
+            <mass value="0.514"/>
             <origin xyz="0.2990 0.1954 0.2118" rpy=" 0 0 0"/>
             <inertia
-                ixx="0.0001" ixy="0" ixz="0"
-                iyy="0.0001" iyz="0"
-                izz="0.0001"
+                ixx="3.125" ixy="0" ixz="0"
+                iyy="4.509" iyz="0"
+                izz="3.125"
             />
         </inertial>
@@ -289,5 +289,5 @@
         <child link="right_wheel_medium"/>
         <axis xyz="0.0 1.0 0.0"/>
-        <limit effort="1.0" velocity="4.0"/>
+        <limit effort="100.0" velocity="15.0"/>
     </joint>
     <link name="right_wheel_medium">
@@ -305,10 +305,10 @@
         </collision>
         <inertial>
-            <mass value="0.0001"/>
+            <mass value="0.514"/>
             <origin xyz="0.2990 0.1954 0.2118" rpy=" 0 0 0"/>
             <inertia
-                ixx="0.0001" ixy="0" ixz="0"
-                iyy="0.0001" iyz="0"
-                izz="0.0001"
+                ixx="3.125" ixy="0" ixz="0"
+                iyy="4.509" iyz="0"
+                izz="3.125"
             />
         </inertial>
@@ -319,5 +319,5 @@
         <child link="right_wheel_back"/>
         <axis xyz="0.0 1.0 0.0"/>
-        <limit effort="1.0" velocity="4.0"/>
+        <limit effort="100.0" velocity="15.0"/>
     </joint>
     <link name="right_wheel_back">
@@ -335,10 +335,10 @@
         </collision>
         <inertial>
-            <mass value="0.0001"/>
+            <mass value="0.514"/>
             <origin xyz="0.2990 0.1954 0.2118" rpy=" 0 0 0"/>
             <inertia
-                ixx="0.0001" ixy="0" ixz="0"
-                iyy="0.0001" iyz="0"
-                izz="0.0001"
+                ixx="3.125" ixy="0" ixz="0"
+                iyy="4.509" iyz="0"
+                izz="3.125"
             />
         </inertial>
@@ -349,5 +349,5 @@
         <child link="left_wheel_front"/>
         <axis xyz="0.0 1.0 0.0"/>
-        <limit effort="100.0" velocity="4.0"/>
+        <limit effort="100.0" velocity="15.0"/>
     </joint>
     <link name="left_wheel_front">
@@ -365,10 +365,10 @@
         </collision>
         <inertial>
-            <mass value="0.0001"/>
+            <mass value="0.514"/>
             <origin xyz="0.2990 0.1954 0.2118" rpy=" 0 0 0"/>
             <inertia
-                ixx="0.0001" ixy="0" ixz="0"
-                iyy="0.0001" iyz="0"
-                izz="0.0001"
+                ixx="3.125" ixy="0" ixz="0"
+                iyy="4.509" iyz="0"
+                izz="3.125"
             />
         </inertial>
@@ -379,5 +379,5 @@
         <child link="left_wheel_medium"/>
         <axis xyz="0.0 1.0 0.0"/>
-        <limit effort="1.0" velocity="4.0"/>
+        <limit effort="100.0" velocity="15.0"/>
     </joint>
     <link name="left_wheel_medium">
@@ -395,10 +395,10 @@
         </collision>
         <inertial>
-            <mass value="0.0001"/>
+            <mass value="0.514"/>
             <origin xyz="0.2990 0.1954 0.2118" rpy=" 0 0 0"/>
             <inertia
-                ixx="0.0001" ixy="0" ixz="0"
-                iyy="0.0001" iyz="0"
-                izz="0.0001"
+                ixx="3.125" ixy="0" ixz="0"
+                iyy="4.509" iyz="0"
+                izz="3.125"
             />
         </inertial>
@@ -409,5 +409,5 @@
         <child link="left_wheel_back"/>
         <axis xyz="0.0 1.0 0.0"/>
-        <limit effort="1.0" velocity="4.0"/>
+        <limit effort="100.0" velocity="15.0"/>
     </joint>
     <link name="left_wheel_back">
@@ -425,10 +425,10 @@
         </collision>
         <inertial>
-            <mass value="0.0001"/>
+            <mass value="0.514"/>
             <origin xyz="0.2990 0.1954 0.2118" rpy=" 0 0 0"/>
             <inertia
-                ixx="0.0001" ixy="0" ixz="0"
-                iyy="0.0001" iyz="0"
-                izz="0.0001"
+                ixx="3.125" ixy="0" ixz="0"
+                iyy="4.509" iyz="0"
+                izz="3.125"
             />
         </inertial>
@@ -479,6 +479,10 @@
         <inertial>
             <origin xyz="0.0 0.0 0.0" rpy="0.0 0.0 0.0"/>
-            <mass value="0.001"/>
-            <inertia ixx="0.001" ixy="0.0" ixz="0.0" iyy="0.001" iyz="0.0" izz="0.001"/>
+            <mass value="0.253"/>
+            <inertia
+                ixx="121.495" ixy="0.026" ixz="-8.296"
+                iyy="1504.113" iyz="0.257"
+                izz="1498.187"
+            />
         </inertial>
     </link>
